File: Hardware/VNA.brd (EAGLE design)
At the start: 161 x 100 mm, 484 parts, among them IC1 ADL5801, IC10 LT5560, IC11 THS4521IDGKR, IC12 MCP33131D-10-E/MS, IC13 SI5351C, IC14 MAX2871, IC15 NCP702-3.3, IC16 RFSW6042, IC17 AP2114H, IC18 RFSW6042, IC19 MAX2871, IC2 LT5560, IC20 NCP702-3.3, IC21 AP2114H, IC22 QPC6324, IC23 RFSA3714, IC24 TRF37A73, IC25 QPC6324, IC26 QPC6324, IC27 QPC6324, IC28 LDL212PU50R, IC29 LDL212PU50R, IC3 THS4521IDGKR, IC30 LDL212PU50R, IC31 LDL212PU50R, IC32 TPS65265, IC34 NCP702-1.8, IC35 NCP702-1.8, IC36 NCP702-1.8, IC37 ADL5801, IC4 MCP33131D-10-E/MS, IC5 ADL5801, IC6 LT5560, IC7 THS4521IDGKR, IC8 MCP33131D-10-E/MS, IC9 STM32G431KB, J1 AMPHENOL_132289, J2 AMPHENOL_132289, J3 DCJ0202, J4 DX07S016JA1R1500, Q1 FA-128 26MHz, T1 B012-617DB-1-63-B331, T2 B012-617DB-1-63-B331, T3 B012-617DB-1-63-B331, U2 6SLX9TQG144, U4 W25Q16BVSN, X4 MINI-USB-SCHIELD-32005-301, X5 10MHz out, X6 10MHz in

Commit message: Placement
Parts:
- removed C167: 1u, VNA:C0603
- added C221, C223: 56p, rcl:C0402
- added C222: 180p, rcl:C0402
- added L19, L20: 330n, rf:R0402
- added L4, L5: Ferrite, rf:R0402
- moved R89 325.7 mm to (128.0, 13.9)
- moved T3 318.8 mm to (167.0, 15.4)
- moved J1 318.8 mm to (128.5, 0.00), turned to 90 degrees
- moved R125 318.6 mm to (127.9, 9.40)
- moved R123 318.5 mm to (129.3, 12.8)
- moved R126 314.9 mm to (129.2, 8.30)
- moved R124 312.9 mm to (128.6, 11.1), turned to 90 degrees
- moved R122 285.3 mm to (152.1, 37.4), turned to 270 degrees
- moved T1 284.9 mm to (133.7, 17.0), turned to 270 degrees
- moved R121 279.2 mm to (148.3, 37.4), turned to 270 degrees
- moved C199 260.9 mm to (212.1, 26.1), turned to 90 degrees
- moved C198 259.5 mm to (212.1, 23.7), turned to 270 degrees
- moved R116 255.4 mm to (159.1, 12.3)
- moved C218 254.5 mm to (162.6, 19.2)
- moved R41 254.3 mm to (154.4, 12.8), turned to 180 degrees
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Connections:
- new net N$235: C155.1, IC25.20, L5.1
- new net N$51: C154.1, IC27.20, L4.2
- new net N$57: C222.1, L19.1, L20.2
- new net REFLO3: C221.1, L19.2, R73.1, R74.1
- net +3V3: now also L4.1, L5.2
- net +5V/4: no longer C167.2
- net GND: now also C221.2, C222.2, C223.2, IC26.16, IC27.17, T3.4; no longer C167.1, IC26.17, IC27.16, T3.2
- net LO1_REF: now also IC13.17; no longer IC13.9
- net N$10: now also T1.2; no longer T1.4
- net N$155: now also IC27.3; no longer IC27.8
- net N$156: no longer C154.1, C155.1, IC25.20, IC27.20
- net N$157: now also C223.1, L20.1; no longer R73.1, R74.1
- net N$160: now also IC13.9; no longer IC13.17
- net N$4: now also T1.6; no longer T1.3
- net N$5: now also T1.4; no longer T1.2
- net N$61: now also T3.6; no longer T3.3
- net N$68: now also T3.3; no longer T3.6
- net N$69: now also T3.2; no longer T3.4
- net N$9: now also T1.3; no longer T1.6
- net PORT1LO2: now also C100.1, L34.2; no longer C97.1, L32.2
- net PORT1SRC: now also IC26.3; no longer IC26.13
- net PORT1_SELECT: now also IC26.17; no longer IC26.16
- net PORT2LO1: now also IC19.14, R65.1; no longer IC19.13, R62.1
- net PORT2LO2: now also C97.1, L32.2; no longer C100.1, L34.2
- net PORT2SRC: now also IC27.8; no longer IC27.3
- net PORT2_SELECT: now also IC27.16; no longer IC27.17
- net REFLO1: now also IC19.13, R62.1; no longer IC19.14, R65.1
Routing:
- net N$147: track 0.00 -> 1.30 mm
- net PORT1LO1: track 0.00 -> 1.30 mm, vias 0 -> 1
- net PORT2LO1: track 0.00 -> 1.17 mm, vias 0 -> 1
- net REFLO1: track 0.00 -> 1.17 mm, vias 0 -> 1
- net SDA: track 0.00 -> 1.04 mm, vias 0 -> 1
- net SCL: track 0.00 -> 1.04 mm, vias 0 -> 1
- net N$115: track 0.00 -> 1.03 mm, vias 0 -> 1
- net N$64: track 0.00 -> 0.96 mm, vias 0 -> 1
- net LO1_MUX: track 0.00 -> 0.93 mm, vias 0 -> 1
- net SOURCE_MUX: track 0.00 -> 0.86 mm, vias 0 -> 1
Other:
- board size 161 x 100 mm -> 239 x 100 mm

Commit message: Placing/routing
Parts:
- added R132, R133, R134: 10k, rcl:R0402
- added R135, R136: 22, rcl:R0402
- J4: value DX07S016JA1R1500 -> TYPE-C16P(073); device custom-connectors:SJ121836 -> custom-connectors:TYPE-C16P
- moved X6 272.1 mm to (220.8, 103.9), turned to 270 degrees
- moved X5 268.1 mm to (231.8, 100.0), turned to 270 degrees
- moved J4 203.9 mm to (182.3, 92.9), turned to 180 degrees
- moved D2 191.0 mm to (171.7, 89.9)
- moved R90 187.0 mm to (211.1, 72.1), flipped to the top
- moved IC9 173.9 mm to (175.2, 75.0), turned to 90 degrees
- moved R95 172.3 mm to (198.0, 70.6), flipped to the top
- moved R114 147.5 mm to (130.0, 17.0)
- moved R112 146.6 mm to (166.4, 67.9), flipped to the top, turned to 0 degrees
- moved C200 145.6 mm to (132.4, 17.6), turned to 270 degrees
- moved C212 144.3 mm to (125.2, 16.3)
- moved R11 141.7 mm to (125.2, 17.5), turned to 180 degrees
- moved L42 141.6 mm to (180.0, 39.0), flipped to the top, turned to 180 degrees
- moved C202 140.7 mm to (125.2, 18.7), turned to 180 degrees
- moved C201 140.5 mm to (125.2, 22.6), turned to 180 degrees
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Connections:
- removed net BAND_SELECT: IC22.16, U2.P22
- removed net N$215: R14.2, U2.P105
- removed net N$216: R26.2, U2.P104
- removed net N$219: R106.2, U2.P85
- removed net N$220: R107.2, U2.P82
- removed net N$221: R108.2, U2.P75
- removed net N$34: IC2.3, L3.1, R34.1, R36.1
- removed net N$65: IC2.4, L11.1, R35.1, R36.2
- removed net PORT1MIX_EN: R112.2, U2.P137
- removed net PORT1_SELECT: IC25.16, IC26.17
- removed net PORT2MIX_EN: R111.2, U2.P44
- removed net PORT2_SELECT: IC25.17, IC27.16
- removed net PORT_SELECT: U2.P23
- removed net REFMIX_EN: R113.2, U2.P35
- new net HIGHBAND_SELECT: IC22.17, U2.P21
- new net LOWBAND_SELECT: IC22.16, U2.P17
- new net N$224: R135.2, U2.P41
- new net PORT1SWITCH: IC26.17, U2.P142
- new net PORT2SWITCH: IC27.17, U2.P40
- new net PORTSWITCH1: IC25.16, U2.P6
- new net PORTSWITCH2: IC25.17, U2.P7
- net +3V3: now also R112.2, R132.2, R133.2
- net AMP_PWDN: now also U2.P8; no longer U2.P24
- net ATT_D0: now also U2.P16; no longer U2.P34
- net ATT_D1: now also U2.P15; no longer U2.P33
- net ATT_D2: now also U2.P14; no longer U2.P32
- net ATT_D3: now also U2.P12; no longer U2.P30
- net ATT_D4: now also U2.P11; no longer U2.P29
- net ATT_D5: now also U2.P10; no longer U2.P27
- net ATT_D6: now also U2.P9; no longer U2.P26
- net FILT_IN_C1: now also U2.P26; no longer U2.P15
- net FILT_IN_C2: now also U2.P24; no longer U2.P16
- net FILT_OUT_C1: now also U2.P22; no longer U2.P21
- net FILT_OUT_C2: now also U2.P23; no longer U2.P17
- net FPGA_RESET: no longer U2.P48
- net GND: now also IC23.10, IC23.11, IC23.12, IC23.13, IC23.15, IC23.25, IC23.4, IC23.6, IC23.7, IC23.8, IC23.9, IC27.16, R134.1; no longer IC27.17, J4.BODY1, J4.BODY2, R112.1
- net LO1_CE: now also U2.P55; no longer U2.P138
- net LO1_CLK: now also U2.P47; no longer U2.P141
- net LO1_LD: now also U2.P45; no longer U2.P142
- net LO1_LE: now also U2.P51; no longer U2.P139
- net LO1_MOSI: now also U2.P48; no longer U2.P140
- net LO1_MUX: now also U2.P56; no longer U2.P144
- net LO1_RF_EN: now also U2.P46; no longer U2.P143
- net MCU_AUX1: no longer U2.P55
- net MCU_AUX2: no longer U2.P51
- net MCU_AUX3: no longer U2.P50
- net MCU_INTR: no longer U2.P57
- net MCU_MISO: no longer U2.P61
- net MCU_MOSI: no longer U2.P59
- net MCU_NSS: no longer U2.P58
- net MCU_SCK: no longer U2.P56
- net N$186: now also J4.8
- net N$189: now also J4.5, J4.7; no longer J4.8
- net N$198: now also U2.P50; no longer U2.P14
- net N$217: now also IC2.4, L11.1, R34.1, R36.1; no longer R42.2, U2.P99
- net N$218: now also IC2.3, L3.1, R35.1, R36.2; no longer R105.2, U2.P94
- net N$228: now also R136.2, U2.P43; no longer IC23.10, IC23.11, IC23.12, IC23.13, IC23.15, IC23.25, IC23.4, IC23.6, IC23.7, IC23.8, IC23.9
- net N$233: now also J4.4; no longer J4.3
- net N$234: now also J4.10; no longer J4.9
- net PORT1LO1: now also IC19.13, R62.1; no longer IC19.12, R63.1
- net PORT1LO2: now also C103.1, L36.2; no longer C100.1, L34.2
- net PORT1MIX1_EN: now also R133.1, U2.P141
- net PORT1MIX2_EN: now also R134.2, U2.P140
- net PORT1_CONVSTART: now also U2.P139; no longer U2.P134
- net PORT1_SCLK: now also U2.P137; no longer U2.P132
- net PORT1_SDO: now also U2.P138; no longer U2.P133
- net PORT2MIX1_EN: now also R112.1, U2.P58
- net PORT2MIX2_EN: now also R111.2, U2.P57
- net PORT2_CONVSTART: now also U2.P44; no longer U2.P47
- net PORT2_SCLK: now also R135.1; no longer U2.P45
- net PORT2_SDO: now also R136.1; no longer U2.P46
- net REFLO1: now also IC19.12, R63.1; no longer IC19.13, R62.1
- net REFLO2: now also C100.1, L34.2; no longer C103.1, L36.2
- net REFMIX1_EN: now also R132.1, U2.P144
- net REFMIX2_EN: now also R113.2, U2.P143
- net REF_CONVSTART: now also U2.P5; no longer U2.P43
- net REF_SCLK: now also U2.P1; no longer U2.P40
- net REF_SDO: now also U2.P2; no longer U2.P41
- net SCL: no longer U2.P6
- net SDA: no longer U2.P9
- net SOURCE_CE: now also U2.P27; no longer U2.P1
- net SOURCE_CLK: now also U2.P32; no longer U2.P7
- net SOURCE_LD: now also U2.P35; no longer U2.P10
- net SOURCE_LE: now also U2.P29; no longer U2.P2
- net SOURCE_MOSI: now also U2.P30; no longer U2.P5
- net SOURCE_MUX: now also U2.P33; no longer U2.P8
- net SOURCE_RF_EN: now also U2.P34; no longer U2.P11
Routing:
- net GND: track 0.00 -> 159.6 mm, vias 0 -> 365
- net PORT1LO2: track 0.00 -> 120.1 mm, vias 0 -> 2
- net PORT1LO1: track 1.30 -> 112.2 mm, vias 1 -> 2
- net +5V/3: track 0.00 -> 101.7 mm, vias 0 -> 10
- net +5V/1: track 0.00 -> 100.9 mm, vias 0 -> 12
- net REFLO1: track 1.17 -> 83.6 mm, vias 1 -> 2
- net REFLO2: track 0.00 -> 78.6 mm, vias 0 -> 2
- net PORTSWITCH2: track 0.00 -> 71.0 mm, vias 0 -> 3
- net PORTSWITCH1: track 0.00 -> 70.9 mm, vias 0 -> 3
- net PORT1SWITCH: track 0.00 -> 62.2 mm, vias 0 -> 3
- net REFMIX1_EN: track 0.00 -> 61.1 mm, vias 0 -> 3
- net ATT_D5: track 0.00 -> 60.2 mm, vias 0 -> 2
- net AMP_PWDN: track 0.00 -> 59.9 mm, vias 0 -> 2
- net ATT_D3: track 0.00 -> 59.2 mm, vias 0 -> 2
- net ATT_D2: track 0.00 -> 59.1 mm, vias 0 -> 2
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- added copper zone on layer 2, net GND

Commit message: Placing/routing
Parts:
- removed JP1: (no value), VNA:1X06
- removed JTAG: (no value), VNA:ML10
- added JP2: (no value), pinhead:1X10/90
- moved R90 140.8 mm to (70.3, 71.4), turned to 0 degrees
- moved R95 128.5 mm to (69.5, 69.8), turned to 0 degrees
- moved R111 123.3 mm to (49.1, 68.0), turned to 180 degrees
- moved R93 118.5 mm to (48.5, 58.9)
- moved C204 118.3 mm to (41.1, 52.4)
- moved TP19 118.1 mm to (79.9, 29.0)
- moved R135 118.0 mm to (49.2, 60.2)
- moved L5 118.0 mm to (64.3, 4.50), turned to 90 degrees
- moved R112 117.3 mm to (49.1, 69.2)
- moved TP16 117.3 mm to (76.0, 52.0)
- moved L39 117.2 mm to (73.3, 57.2)
- moved C128 117.2 mm to (73.3, 58.7)
- moved C126 117.1 mm to (79.2, 54.9)
- moved C123 117.1 mm to (80.6, 57.9)
- moved C124 117.1 mm to (75.5, 57.9)
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Connections:
- removed net N$183: JTAG.1, U2.P109
- removed net N$222: R109.2, U2.P118
- new net N$34: JP2.1, U2.P109
- new net N$65: JP2.2, U2.P106
- net +3V3: now also JP2.5; no longer JP1.1, JTAG.4
- net GND: now also JP2.7; no longer JP1.3, JTAG.10, JTAG.2
- net LO1_CE: now also U2.P45; no longer U2.P55
- net LO1_CLK: now also U2.P48; no longer U2.P47
- net LO1_LD: now also U2.P56; no longer U2.P45
- net LO1_LE: now also U2.P46; no longer U2.P51
- net LO1_MOSI: now also U2.P47; no longer U2.P48
- net LO1_MUX: now also U2.P51; no longer U2.P56
- net LO1_RF_EN: now also U2.P55; no longer U2.P46
- net N$165: now also JP2.3, U2.P110; no longer JTAG.3, U2.P106
- net N$173: now also JP2.4; no longer JTAG.5
- net N$175: now also R109.2; no longer JTAG.9, U2.P110
- net N$190: now also JP2.6; no longer JP1.2
- net N$191: now also JP2.8; no longer JP1.4
- net N$192: now also JP2.9; no longer JP1.5
- net N$193: now also JP2.10; no longer JP1.6
Routing:
- net +3V3: track 20.4 -> 288.0 mm, vias 1 -> 19
- net GND: track 159.6 -> 384.8 mm, vias 365 -> 707
- net +5V/2: track 0.00 -> 117.5 mm, vias 0 -> 9
- net PORT2MIX2_EN: track 0.00 -> 109.1 mm, vias 0 -> 3
- net PORT2MIX1_EN: track 0.00 -> 91.7 mm, vias 0 -> 2
- net PORT2SWITCH: track 0.00 -> 90.6 mm, vias 0 -> 4
- net +5V/4: track 0.00 -> 86.5 mm, vias 0 -> 7
- net LO1_LE: track 0.00 -> 81.4 mm, vias 0 -> 2
- net LO1_CLK: track 0.00 -> 80.5 mm, vias 0 -> 2
- net LO1_CE: track 0.00 -> 80.4 mm, vias 0 -> 2
- net N$228: track 0.00 -> 79.8 mm, vias 0 -> 2
- net LO1_MOSI: track 0.00 -> 78.5 mm, vias 0 -> 2
- net PORT2_CONVSTART: track 0.00 -> 78.1 mm, vias 0 -> 2
- net LO1_MUX: track 0.93 -> 77.4 mm, vias 1 -> 2
- net LO1_RF_EN: track 0.00 -> 76.3 mm, vias 0 -> 2
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Other:
- board size 239 x 100 mm -> 122 x 96 mm
- board text removed: "+12V IN"
- board text removed: "+1V8"
- board text removed: "+5V"
- board text removed: "+6V"
- board text removed: "05/2020"
- board text removed: "1MHz-6GHz VNA"
- board text removed: "GND"
- board text removed: "JTAG"
- board text removed: "Ref IN"
- board text removed: "Ref OUT"
- board text removed: "SWD/TX"
- board text removed: "github.com/jankae/VNA"

Commit message: Placing/routing
Parts:
- added C167, C224, C225, C226, C227: 100n, rcl:C0402
- C168: value 1u -> 1u/25V
- C176: value 510p -> 1n
- C179: value DNP -> 8p2
- C187: value 1n -> 510p
- C188: value 8p2 -> DNP
- JP2: value (none) -> DNP
- R82: value 30k -> 16k
- R84: value 45k3 -> 20k
- R85: value 16k -> 30k
- R87: value 20k -> 45k3
- X4: value MINI-USB-SCHIELD-32005-301 -> DNP
- moved J4 34.0 mm to (64.0, 88.1)
- moved J3 33.8 mm to (76.0, 85.5)
- moved JP2 33.0 mm to (32.7, 93.6)
- moved X4 32.8 mm to (52.5, 90.3)
- moved X5 27.6 mm to (95.0, 95.9), turned to 270 degrees
- moved X6 26.1 mm to (111.0, 95.9), turned to 270 degrees
- moved TP5 25.7 mm to (11.3, 62.4)
- moved D1 24.8 mm to (76.0, 79.0), turned to 180 degrees
- moved C65 21.5 mm to (95.0, 90.5), turned to 90 degrees
- moved D2 20.0 mm to (76.0, 75.0), turned to 180 degrees
- moved C107 19.1 mm to (111.0, 90.5), turned to 270 degrees
- moved C189 16.7 mm to (75.5, 70.0), turned to 90 degrees
- moved C190 16.7 mm to (73.0, 70.0), turned to 90 degrees
- moved L55 16.6 mm to (79.7, 70.3), turned to 180 degrees
- moved C208 15.4 mm to (21.4, 66.6), turned to 180 degrees
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Connections:
- new net MCU_FPGA_UNUSED1: IC9.30, U2.P79
- new net MCU_FPGA_UNUSED2: IC9.26, U2.P80
- new net MCU_FPGA_UNUSED3: IC9.25, U2.P81
- new net N$183: C180.1, C184.1, C188.1, L54.P$2, L55.P$1, R87.2
- new net N$215: R14.2, U2.P82
- new net N$216: R26.2, U2.P83
- new net N$219: R42.2, U2.P84
- new net N$220: R105.2, U2.P85
- new net N$221: R106.2, U2.P87
- new net N$222: R107.2, U2.P88
- net +3V3: now also C224.1, C225.1, C226.1, C227.1
- net FPGA_RESET: now also U2.P72
- net GND: now also C167.2, C224.2, C225.2, C226.2, C227.2
- net MCU_AUX1: now also U2.P78
- net MCU_AUX2: now also U2.P74
- net MCU_AUX3: now also U2.P75
- net MCU_INTR: now also U2.P59
- net MCU_MISO: now also U2.P62
- net MCU_MOSI: now also U2.P61
- net MCU_NSS: now also U2.P67
- net MCU_SCK: now also U2.P66
- net N$175: now also U2.P92
- net N$179: now also R108.2, U2.P93; no longer C169.1, C172.1, C179.1, L53.P$2, L55.P$1, R84.2
- net POWER_GOOD: now also IC9.8
- net VCCINT: now also C167.1, C169.1, C172.1, C179.1, L53.P$2, R84.2; no longer C180.1, C184.1, C188.1, L54.P$2, R87.2
Routing:
- net +3V3: track 288.0 -> 410.6 mm, vias 19 -> 62
- net SDA: track 1.04 -> 73.3 mm, vias 1 -> 4
- net GND: track 384.8 -> 451.3 mm, vias 707 -> 785
- net SCL: track 1.04 -> 65.7 mm, vias 1 -> 3
- net N$103: track 1.49 -> 63.8 mm, vias 1 -> 3
- net N$108: track 0.00 -> 59.2 mm, vias 0 -> 3
- net VCCINT: track 8.27 -> 57.9 mm, vias 0 -> 11
- net POWER_GOOD: track 0.00 -> 37.4 mm, vias 0 -> 2
- net MCU_INTR: track 0.00 -> 34.0 mm
- net N$216: track 0.00 -> 33.2 mm, vias 0 -> 2
- net N$215: track 0.00 -> 33.2 mm, vias 0 -> 2
- net N$190: track 0.00 -> 32.5 mm
- net MCU_MOSI: track 0.00 -> 32.4 mm
- net MCU_MISO: track 0.00 -> 31.2 mm
- net MCU_SCK: track 0.00 -> 30.6 mm
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- added copper zone on layer 1, net +12V
- added copper zone on layer 16, net +12V
- added copper zone on layer 15, net +3V3
- added copper zone on layer 1, net GND
- added copper zone on layer 15, net GND
- added copper zone on layer 15, net N$163
- added copper zone on layer 1, net N$169
- added copper zone on layer 1, net N$171
- added copper zone on layer 1, net N$181
- added copper zone on layer 15, net VCCINT

Commit message: Routing completed
Parts:
- added C228: 100n, rcl:C0402
- added R137, R138, R139, R140, R141, R142, R143, R144, R145, R146, R147: 0, rcl:R0402
- IC9: value STM32G431KB -> STM32G431CB; device custom-ic:QFN50P500X500X100-33T345N -> custom-ic:QFN50P700X700X60-49T560N
- R91: value 22 -> 0
- moved TP5 16.9 mm to (28.0, 60.0)
- moved C224 14.6 mm to (50.2, 64.2), turned to 180 degrees
- moved TP3 12.4 mm to (28.0, 62.0)
- moved U4 11.3 mm to (55.4, 65.2)
- moved TP1 7.36 mm to (28.0, 64.0)
- moved TP6 6.99 mm to (28.0, 66.0)
- moved C192 3.04 mm to (60.5, 73.0), turned to 180 degrees
- moved R91 2.93 mm to (53.9, 73.7), turned to 180 degrees
- moved R95 2.02 mm to (66.0, 84.3), turned to 90 degrees
- moved C191 1.84 mm to (70.0, 79.7), turned to 90 degrees
- moved R90 1.66 mm to (67.3, 84.3), turned to 90 degrees
- moved IC9 1.52 mm to (65.1, 77.8)
Connections:
- removed net FLACH_MOSI: U2.P64, U4.5
- removed net FLASH_CLK: U2.P70, U4.6
- removed net FLASH_CS: U2.P38, U4.1
- removed net FLASH_MISO: R91.1, U4.2
- removed net MCU_NSS: IC9.9, U2.P67
- removed net N$190: IC9.24, JP2.6
- removed net N$191: IC9.23, JP2.8
- removed net N$194: R92.1, U2.P71
- removed net N$195: R93.1, U2.P39
- removed net N$196: R94.1, U2.P37
- new net FPGA_CCLK: R146.2, R91.2, U2.P70
- new net FPGA_CSO_B: R139.2, U2.P38
- new net FPGA_DIN: R138.2, R147.2, U2.P65
- new net FPGA_DONE: IC9.47, R92.1, U2.P71
- new net FPGA_INIT_B: IC9.6, R93.1, U2.P39
- new net FPGA_M1: R140.1, R141.2, U2.P60
- new net FPGA_MOSI: R137.2, U2.P64
- new net FPGA_PROGRAM_B: IC9.19, R94.1, U2.P37
- new net MCU_FLASH_CS: IC9.17, R142.1
- new net MCU_FPGA_CCLK: IC9.28, R146.1
- new net MCU_FPGA_DIN: IC9.26, R147.1
- new net MCU_FPGA_NSS: IC9.12, U2.P67
- new net N$237: R137.1, R144.2, U4.5
- new net N$240: R138.1, R143.2, U4.2
- new net N$241: R139.1, R142.2, U4.1
- new net SWCLK: IC9.37, JP2.6
- new net SWDIO: IC9.36, JP2.8
- net +3V3: now also C228.1, IC9.20, IC9.21, IC9.23, IC9.35, IC9.48, R141.1; no longer IC9.15, IC9.17
- net FPGA_RESET: now also IC9.45; no longer IC9.6
- net GND: now also C228.2, IC9.46, IC9.49, R140.2; no longer IC9.14, IC9.16, IC9.31, IC9.32, IC9.33, U2.P60
- net MCU_AUX1: now also IC9.9; no longer IC9.2
- net MCU_AUX2: now also IC9.10; no longer IC9.3
- net MCU_AUX3: now also IC9.11; no longer IC9.5
- net MCU_FPGA_UNUSED1: now also IC9.43; no longer IC9.30
- net MCU_FPGA_UNUSED2: now also IC9.41; no longer IC9.26
- net MCU_FPGA_UNUSED3: now also IC9.40; no longer IC9.25
- net MCU_INTR: now also IC9.18; no longer IC9.13
- net MCU_MISO: now also IC9.14, R143.1; no longer IC9.11
- net MCU_MOSI: now also IC9.15, R144.1; no longer IC9.12
- net MCU_SCK: now also IC9.13, R145.1; no longer IC9.10
- net N$187: now also IC9.33; no longer IC9.21
- net N$188: now also IC9.34; no longer IC9.22
- net N$192: now also IC9.7; no longer IC9.4
- net N$193: now also IC9.39; no longer IC9.7
- net N$197: now also R145.2, R91.1, U4.6; no longer R91.2, U2.P65
- net N$233: now also IC9.31, IC9.44; no longer IC9.19, IC9.29
- net N$234: now also IC9.32, IC9.42; no longer IC9.20, IC9.27
- net POWER_GOOD: now also IC9.25; no longer IC9.8
- net SCL: now also IC9.16; no longer IC9.18
- net SDA: now also IC9.30; no longer IC9.28
Routing:
- net GND: track 451.3 -> 746.5 mm, vias 785 -> 1555
- net FPGA_PROGRAM_B: track 0.00 -> 40.4 mm, vias 0 -> 2
- net FPGA_INIT_B: track 0.00 -> 33.3 mm, vias 0 -> 2
- net N$190: track 32.5 -> 0.00 mm
- net SWCLK: track 0.00 -> 31.5 mm
- net FLASH_CS: track 30.2 -> 0.00 mm, vias 2 -> 0
- net MCU_NSS: track 29.4 -> 0.00 mm
- net N$191: track 28.1 -> 0.00 mm
- net SWDIO: track 0.00 -> 26.8 mm
- net MCU_FPGA_NSS: track 0.00 -> 26.3 mm, vias 0 -> 2
- net MCU_FLASH_CS: track 0.00 -> 23.4 mm
- net FPGA_CSO_B: track 0.00 -> 22.7 mm, vias 0 -> 2
- net N$163: track 85.0 -> 107.4 mm, vias 18 -> 19
- net FPGA_DONE: track 0.00 -> 20.7 mm
- net FPGA_CCLK: track 0.00 -> 17.8 mm
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
Commit message: Routing + BOM
Parts:
- removed R68: 0, rcl:R0402
- added JP1: DNP, pinhead:2X10
- added LED10: Red, led:CHIPLED_0603
- added R148: 330, rcl:R0402
- C1, C150, C153, C2, C3, C33, C34, C35, C36, C4, C66, C67, C68: value 100n -> 100n/RF
- C121, C132: value 10n -> 100n/RF
- C131: value 10n -> 100n
- C168: value 1u/25V -> 1u
- LED1, LED5, LED6, LED7, LED8, LED9: value (none) -> Green
- LED2, LED3, LED4: value (none) -> Red
- R135, R136, R76, R88, R96: value 22 -> 20
- R137, R138, R139, R140, R91: value 0 -> DNP
- X5: value 10MHz out -> (none)
- X6: value 10MHz in -> (none)
- moved LED1 3.00 mm to (37.6, 82.8)
- moved R110 3.00 mm to (39.1, 82.8)
Connections:
- net N$165 renamed TDI
- net N$173 renamed TMS
- net N$192 renamed NRST
- net N$193 renamed UART_TX
- net N$34 renamed TCK
- net N$65 renamed TDO
- removed net N$158: IC23.5, R68.2
- new net N$190: LED10.C, R148.1
- new net N$191: IC9.38, R148.2
- new net N$194: JP1.2, U2.P134
- new net N$195: JP1.4, U2.P133
- new net N$196: JP1.3, U2.P132
- new net N$242: JP1.6, U2.P131
- new net N$243: JP1.5, U2.P127
- new net N$244: JP1.8, U2.P126
- new net N$245: JP1.7, U2.P124
- new net N$246: JP1.10, U2.P123
- new net N$247: JP1.9, U2.P121
- new net N$248: JP1.12, U2.P120
- new net N$249: JP1.11, U2.P119
- new net N$250: JP1.14, U2.P118
- new net N$251: JP1.13, U2.P117
- new net N$252: JP1.16, U2.P116
- new net N$253: JP1.15, U2.P115
- new net N$254: JP1.18, U2.P114
- new net N$255: JP1.17, U2.P112
- new net N$256: JP1.19, U2.P111
- net +3V3: now also JP1.1, LED10.A
- net GND: now also JP1.20
- net N$144: now also IC23.5; no longer R68.1
Routing:
- net N$191: track 0.00 -> 29.3 mm
- net N$256: track 0.00 -> 25.9 mm
- net N$246: track 0.00 -> 24.5 mm, vias 0 -> 1
- net N$254: track 0.00 -> 24.2 mm
- net N$244: track 0.00 -> 24.1 mm, vias 0 -> 1
- net N$255: track 0.00 -> 23.7 mm
- net N$252: track 0.00 -> 22.8 mm
- net N$250: track 0.00 -> 22.2 mm
- net N$247: track 0.00 -> 21.6 mm, vias 0 -> 1
- net N$248: track 0.00 -> 21.5 mm
- net +3V3: track 410.3 -> 389.2 mm, vias 67 -> 68
- net N$245: track 0.00 -> 21.1 mm, vias 0 -> 1
- net N$243: track 0.00 -> 20.7 mm, vias 0 -> 1
- net N$242: track 0.00 -> 20.7 mm
- net N$253: track 0.00 -> 20.1 mm
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Other:
- board text added: "+12V In"
- board text added: "+1V8"
- board text added: "+5V"
- board text added: "+6V"
- board text added: "GND"
- board text added: "NRST"
- board text added: "Port 1"
- board text added: "Port 2"
- board text added: "Ref In"
- board text added: "Ref Out"
- board text added: "SWCLK"
- board text added: "SWDIO"
- board text added: "TCK"
- board text added: "TDI"
- board text added: "TDO"
- board text added: "TMS"
- board text added: "TX"
