File: Hardware/VNA.sch (EAGLE design)
At the start: 484 parts, among them IC1 ADL5801, IC10 LT5560, IC11 THS4521IDGKR, IC12 MCP33131D-10-E/MS, IC13 SI5351C, IC14 MAX2871, IC15 NCP702-3.3, IC16 RFSW6042, IC17 AP2114H, IC18 RFSW6042, IC19 MAX2871, IC2 LT5560, IC20 NCP702-3.3, IC21 AP2114H, IC22 QPC6324, IC23 RFSA3714, IC24 TRF37A73, IC25 QPC6324, IC26 QPC6324, IC27 QPC6324, IC28 LDL212PU50R, IC29 LDL212PU50R, IC3 THS4521IDGKR, IC30 LDL212PU50R, IC31 LDL212PU50R, IC32 TPS65265, IC34 NCP702-1.8, IC35 NCP702-1.8, IC36 NCP702-1.8, IC37 ADL5801, IC4 MCP33131D-10-E/MS, IC5 ADL5801, IC6 LT5560, IC7 THS4521IDGKR, IC8 MCP33131D-10-E/MS, IC9 STM32G431KB, J1 AMPHENOL_132289, J2 AMPHENOL_132289, J3 DCJ0202, J4 DX07S016JA1R1500, Q1 FA-128 26MHz, T1 B012-617DB-1-63-B331, T2 B012-617DB-1-63-B331, T3 B012-617DB-1-63-B331, U2 6SLX9TQG144, U4 W25Q16BVSN, X4 MINI-USB-SCHIELD-32005-301, X5 10MHz out, X6 10MHz in

Commit message: Placement
Parts:
- removed C167: 1u, VNA:C-EUC0603
- added C221, C223: 56p, rcl:C-EUC0402
- added C222: 180p, rcl:C-EUC0402
- added L19, L20: 330n, rf:INDUCTOR0402
- added L4, L5: Ferrite, rf:INDUCTOR0402
Connections:
- new net N$235: C155.1, IC25.VCC, L5.1
- new net N$51: C154.1, IC27.VCC, L4.2
- new net N$57: C222.1, L19.1, L20.2
- new net REFLO3: C221.1, L19.2, R73.1, R74.1
- net +3V3: now also L4.1, L5.2
- net +5V/4: no longer C167.2
- net GND: now also C221.2, C222.2, C223.2, IC26.CTL2, IC27.CTL1, T3.OUT+; no longer C167.1, IC26.CTL1, IC27.CTL2, T3.IN-
- net LO1_REF: now also IC13.CLK5; no longer IC13.CLK2
- net N$10: now also T1.IN-; no longer T1.OUT+
- net N$155: now also IC27.RF1; no longer IC27.RF_COM
- net N$156: no longer C154.1, C155.1, IC25.VCC, IC27.VCC
- net N$157: now also C223.1, L20.1; no longer R73.1, R74.1
- net N$160: now also IC13.CLK2; no longer IC13.CLK5
- net N$4: now also T1.OUT-; no longer T1.IN+
- net N$5: now also T1.OUT+; no longer T1.IN-
- net N$61: now also T3.OUT-; no longer T3.IN+
- net N$68: now also T3.IN+; no longer T3.OUT-
- net N$69: now also T3.IN-; no longer T3.OUT+
- net N$9: now also T1.IN+; no longer T1.OUT-
- net PORT1LO2: now also C100.1, L34.2; no longer C97.1, L32.2
- net PORT1SRC: now also IC26.RF1; no longer IC26.RF2
- net PORT1_SELECT: now also IC26.CTL1; no longer IC26.CTL2
- net PORT2LO1: now also IC19.RFOUTB_P, R65.1; no longer IC19.RFOUTA_N, R62.1
- net PORT2LO2: now also C97.1, L32.2; no longer C100.1, L34.2
- net PORT2SRC: now also IC27.RF_COM; no longer IC27.RF1
- net PORT2_SELECT: now also IC27.CTL2; no longer IC27.CTL1
- net REFLO1: now also IC19.RFOUTA_N, R62.1; no longer IC19.RFOUTB_P, R65.1
Other:
- note added: "3x110MHz lowpass"
- note added: "40MHz lowpass"
- moved on the sheet: C154, C155, C156, C157, IC26, IC27, L46, R73, R74, R75, T1, T3

Commit message: Placing/routing
Parts:
- added R132, R133, R134: 10k, rcl:R-EU_R0402
- added R135, R136: 22, rcl:R-EU_R0402
- J4: value DX07S016JA1R1500 -> TYPE-C16P(073); device custom-connectors:DX07S016JA1R1500 -> custom-connectors:TYPE-C16P(073)
Connections:
- removed net BAND_SELECT: IC22.CTL2, U2B3.IO_L42P_GCLK25_TRDY2_3
- removed net N$215: R14.2, U2B1.IO_L1P_1
- removed net N$216: R26.2, U2B1.IO_L1N_VREF_1
- removed net N$219: R106.2, U2B1.IO_L43P_GCLK5_1
- removed net N$220: R107.2, U2B1.IO_L45N_1
- removed net N$221: R108.2, U2B1.IO_L74P_AWAKE_1
- removed net N$34: IC2.IN+, L3.1, R34.1, R36.1
- removed net N$65: IC2.IN-, L11.1, R35.1, R36.2
- removed net PORT1MIX_EN: R112.2, U2B0.IO_L4N_0
- removed net PORT1_SELECT: IC25.CTL2, IC26.CTL1
- removed net PORT2MIX_EN: R111.2, U2B2.IO_L62P_D5_2
- removed net PORT2_SELECT: IC25.CTL1, IC27.CTL2
- removed net PORT_SELECT: U2B3.IO_L41N_GCLK26_3
- removed net REFMIX_EN: R113.2, U2B3.IO_L1P_3
- new net HIGHBAND_SELECT: IC22.CTL1, U2B3.IO_L42N_GCLK24_3
- new net LOWBAND_SELECT: IC22.CTL2, U2B3.IO_L43P_GCLK23_3
- new net N$224: R135.2, U2B2.IO_L64P_D8_2
- new net PORT1SWITCH: IC26.CTL1, U2B0.IO_L2P_0
- new net PORT2SWITCH: IC27.CTL1, U2B2.IO_L64N_D9_2
- new net PORTSWITCH1: IC25.CTL2, U2B3.IO_L52P_3
- new net PORTSWITCH2: IC25.CTL1, U2B3.IO_L51N_3
- net +3V3: now also R112.2, R132.2, R133.2
- net AMP_PWDN: now also U2B3.IO_L51P_3; no longer U2B3.IO_L41P_GCLK27_3
- net ATT_D0: now also U2B3.IO_L43N_GCLK22_IRDY2_3; no longer U2B3.IO_L1N_VREF_3
- net ATT_D1: now also U2B3.IO_L44P_GCLK21_3; no longer U2B3.IO_L2P_3
- net ATT_D2: now also U2B3.IO_L44N_GCLK20_3; no longer U2B3.IO_L2N_3
- net ATT_D3: now also U2B3.IO_L49P_3; no longer U2B3.IO_L36P_3
- net ATT_D4: now also U2B3.IO_L49N_3; no longer U2B3.IO_L36N_3
- net ATT_D5: now also U2B3.IO_L50P_3; no longer U2B3.IO_L37P_3
- net ATT_D6: now also U2B3.IO_L50N_3; no longer U2B3.IO_L37N_3
- net FILT_IN_C1: now also U2B3.IO_L37N_3; no longer U2B3.IO_L44P_GCLK21_3
- net FILT_IN_C2: now also U2B3.IO_L41P_GCLK27_3; no longer U2B3.IO_L43N_GCLK22_IRDY2_3
- net FILT_OUT_C1: now also U2B3.IO_L42P_GCLK25_TRDY2_3; no longer U2B3.IO_L42N_GCLK24_3
- net FILT_OUT_C2: now also U2B3.IO_L41N_GCLK26_3; no longer U2B3.IO_L43P_GCLK23_3
- net FPGA_RESET: no longer U2B2.IO_L48P_D7_2
- net GND: now also IC23.GND, IC27.CTL2, R134.1; no longer IC27.CTL1, R112.1
- net LO1_CE: now also U2B2.IO_L30N_GCLK0_USERCCLK_2; no longer U2B0.IO_L4P_0
- net LO1_CLK: now also U2B2.IO_L48N_RDWR_B_VREF_2; no longer U2B0.IO_L2N_0
- net LO1_LD: now also U2B2.IO_L49N_D4_2; no longer U2B0.IO_L2P_0
- net LO1_LE: now also U2B2.IO_L31P_GCLK31_D14_2; no longer U2B0.IO_L3N_0
- net LO1_MOSI: now also U2B2.IO_L48P_D7_2; no longer U2B0.IO_L3P_0
- net LO1_MUX: now also U2B2.IO_L30P_GCLK1_D13_2; no longer U2B0.IO_L1P_HSWAPEN_0
- net LO1_RF_EN: now also U2B2.IO_L49P_D3_2; no longer U2B0.IO_L1N_VREF_0
- net MCU_AUX1: no longer U2B2.IO_L30N_GCLK0_USERCCLK_2
- net MCU_AUX2: no longer U2B2.IO_L31P_GCLK31_D14_2
- net MCU_AUX3: no longer U2B2.IO_L31N_GCLK30_D15_2
- net MCU_INTR: no longer U2B2.IO_L14N_D12_2
- net MCU_MISO: no longer U2B2.IO_L12N_D2_MISO3_2
- net MCU_MOSI: no longer U2B2.IO_L13N_D10_2
- net MCU_NSS: no longer U2B2.IO_L14P_D11_2
- net MCU_SCK: no longer U2B2.IO_L30P_GCLK1_D13_2
- net N$186: now also J4.D+1
- net N$189: now also J4.D-1
- net N$198: now also U2B2.IO_L31N_GCLK30_D15_2; no longer U2B3.IO_L44N_GCLK20_3
- net N$217: now also IC2.IN-, L11.1, R34.1, R36.1; no longer R42.2, U2B1.IO_L33N_1
- net N$218: now also IC2.IN+, L3.1, R35.1, R36.2; no longer R105.2, U2B1.IO_L40N_GCLK10_1
- net N$228: now also R136.2, U2B2.IO_L62N_D6_2; no longer IC23.GND
- net PORT1LO1: now also IC19.RFOUTA_N, R62.1; no longer IC19.RFOUTA_P, R63.1
- net PORT1LO2: now also C103.1, L36.2; no longer C100.1, L34.2
- net PORT1MIX1_EN: now also R133.1, U2B0.IO_L2N_0
- net PORT1MIX2_EN: now also R134.2, U2B0.IO_L3P_0
- net PORT1_CONVSTART: now also U2B0.IO_L3N_0; no longer U2B0.IO_L34P_GCLK19_0
- net PORT1_SCLK: now also U2B0.IO_L4N_0; no longer U2B0.IO_L35P_GCLK17_0
- net PORT1_SDO: now also U2B0.IO_L4P_0; no longer U2B0.IO_L34N_GCLK18_0
- net PORT2MIX1_EN: now also R112.1, U2B2.IO_L14P_D11_2
- net PORT2MIX2_EN: now also R111.2, U2B2.IO_L14N_D12_2
- net PORT2_CONVSTART: now also U2B2.IO_L62P_D5_2; no longer U2B2.IO_L48N_RDWR_B_VREF_2
- net PORT2_SCLK: now also R135.1; no longer U2B2.IO_L49N_D4_2
- net PORT2_SDO: now also R136.1; no longer U2B2.IO_L49P_D3_2
- net REFLO1: now also IC19.RFOUTA_P, R63.1; no longer IC19.RFOUTA_N, R62.1
- net REFLO2: now also C100.1, L34.2; no longer C103.1, L36.2
- net REFMIX1_EN: now also R132.1, U2B0.IO_L1P_HSWAPEN_0
- net REFMIX2_EN: now also R113.2, U2B0.IO_L1N_VREF_0
- net REF_CONVSTART: now also U2B3.IO_L52N_3; no longer U2B2.IO_L62N_D6_2
- net REF_SCLK: now also U2B3.IO_L83N_VREF_3; no longer U2B2.IO_L64N_D9_2
- net REF_SDO: now also U2B3.IO_L83P_3; no longer U2B2.IO_L64P_D8_2
- net SCL: no longer U2B3.IO_L52P_3
- net SDA: no longer U2B3.IO_L50N_3
- net SOURCE_CE: now also U2B3.IO_L37P_3; no longer U2B3.IO_L83N_VREF_3
- net SOURCE_CLK: now also U2B3.IO_L2N_3; no longer U2B3.IO_L51N_3
- net SOURCE_LD: now also U2B3.IO_L1P_3; no longer U2B3.IO_L50P_3
- net SOURCE_LE: now also U2B3.IO_L36N_3; no longer U2B3.IO_L83P_3
- net SOURCE_MOSI: now also U2B3.IO_L36P_3; no longer U2B3.IO_L52N_3
- net SOURCE_MUX: now also U2B3.IO_L2P_3; no longer U2B3.IO_L51P_3
- net SOURCE_RF_EN: now also U2B3.IO_L1N_VREF_3; no longer U2B3.IO_L49N_3
Other:
- moved on the sheet: D2, R111, R113, U2B3

Commit message: Placing/routing
Parts:
- removed JP1: (no value), VNA:PINHD-1X6
- removed JTAG: (no value), VNA:ML10
- added JP2: (no value), pinhead:PINHD-1X10/90
Connections:
- removed net N$183: JTAG.1, U2BNA.TCK
- removed net N$222: R109.2, U2B0.IO_L63N_SCP6_0
- new net N$34: JP2.1, U2BNA.TCK
- new net N$65: JP2.2, U2BNA.TDO
- net +3V3: now also JP2.5; no longer JP1.1, JTAG.4
- net GND: now also JP2.7; no longer JP1.3, JTAG.10, JTAG.2
- net LO1_CE: now also U2B2.IO_L49N_D4_2; no longer U2B2.IO_L30N_GCLK0_USERCCLK_2
- net LO1_CLK: now also U2B2.IO_L48P_D7_2; no longer U2B2.IO_L48N_RDWR_B_VREF_2
- net LO1_LD: now also U2B2.IO_L30P_GCLK1_D13_2; no longer U2B2.IO_L49N_D4_2
- net LO1_LE: now also U2B2.IO_L49P_D3_2; no longer U2B2.IO_L31P_GCLK31_D14_2
- net LO1_MOSI: now also U2B2.IO_L48N_RDWR_B_VREF_2; no longer U2B2.IO_L48P_D7_2
- net LO1_MUX: now also U2B2.IO_L31P_GCLK31_D14_2; no longer U2B2.IO_L30P_GCLK1_D13_2
- net LO1_RF_EN: now also U2B2.IO_L30N_GCLK0_USERCCLK_2; no longer U2B2.IO_L49P_D3_2
- net N$165: now also JP2.3, U2BNA.TDI; no longer JTAG.3, U2BNA.TDO
- net N$173: now also JP2.4; no longer JTAG.5
- net N$175: now also R109.2; no longer JTAG.9, U2BNA.TDI
- net N$190: now also JP2.6; no longer JP1.2
- net N$191: now also JP2.8; no longer JP1.4
- net N$192: now also JP2.9; no longer JP1.5
- net N$193: now also JP2.10; no longer JP1.6
Other:
- moved on the sheet: U2BNA

Commit message: Placing/routing
Parts:
- added C167, C224, C225, C226, C227: 100n, rcl:C-EUC0402
- C168: value 1u -> 1u/25V
- C176: value 510p -> 1n
- C179: value DNP -> 8p2
- C187: value 1n -> 510p
- C188: value 8p2 -> DNP
- JP2: value (none) -> DNP
- R82: value 30k -> 16k
- R84: value 45k3 -> 20k
- R85: value 16k -> 30k
- R87: value 20k -> 45k3
- X4: value MINI-USB-SCHIELD-32005-301 -> DNP
Connections:
- new net MCU_FPGA_UNUSED1: IC9.PB7/TIM4_CH2/I2C1_SDA/USART1_RX/TIM3_CH4, U2B1.IO_L47P_1
- new net MCU_FPGA_UNUSED2: IC9.PB3/TIM2_CH2/SPI1_SCK/SPI3_SCK/USART2_TX, U2B1.IO_L46N_1
- new net MCU_FPGA_UNUSED3: IC9.PA15/TIM2_CH1/TIM8_CH1/I2C1_SCL/USART2_RX/SPI1_NSS/SPI3_NSS, U2B1.IO_L46P_1
- new net N$183: C180.1, C184.1, C188.1, L54.2, L55.1, R87.2
- new net N$215: R14.2, U2B1.IO_L45N_1
- new net N$216: R26.2, U2B1.IO_L45P_1
- new net N$219: R42.2, U2B1.IO_L43N_GCLK4_1
- new net N$220: R105.2, U2B1.IO_L43P_GCLK5_1
- new net N$221: R106.2, U2B1.IO_L42N_GCLK6_TRDY1_1
- new net N$222: R107.2, U2B1.IO_L42P_GCLK7_1
- net +3V3: now also C224.1, C225.1, C226.1, C227.1
- net FPGA_RESET: now also U2B2.CMPCS_B_2
- net GND: now also C167.2, C224.2, C225.2, C226.2, C227.2
- net MCU_AUX1: now also U2B1.IO_L47N_1
- net MCU_AUX2: now also U2B1.IO_L74N_DOUT_BUSY_1
- net MCU_AUX3: now also U2B1.IO_L74P_AWAKE_1
- net MCU_INTR: now also U2B2.IO_L13N_D10_2
- net MCU_MISO: now also U2B2.IO_L12P_D1_MISO2_2
- net MCU_MOSI: now also U2B2.IO_L12N_D2_MISO3_2
- net MCU_NSS: now also U2B2.IO_L2P_CMPCLK_2
- net MCU_SCK: now also U2B2.IO_L2N_CMPMOSI_2
- net N$175: now also U2B1.IO_L41N_GCLK8_1
- net N$179: now also R108.2, U2B1.IO_L41P_GCLK9_IRDY1_1; no longer C169.1, C172.1, C179.1, L53.2, L55.1, R84.2
- net POWER_GOOD: now also IC9.PA3/TIM2_CH4/USART2_RX/TIM15_CH2
- net VCCINT: now also C167.1, C169.1, C172.1, C179.1, L53.2, R84.2; no longer C180.1, C184.1, C188.1, L54.2, R87.2
Other:
- moved on the sheet: C189, C190, C203, C204, C205, C206, C207, C208, C209, C210, C211, L55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

Commit message: Routing completed
Parts:
- added C228: 100n, rcl:C-EUC0402
- added R137, R138, R139, R140, R141, R142, R143, R144, R145, R146, R147: 0, rcl:R-EU_R0402
- IC9: value STM32G431KB -> STM32G431CB; device custom-ic:STM32G431KB -> custom-ic:STM32G431CB
- R91: value 22 -> 0
Connections:
- removed net FLACH_MOSI: U2B2.IO_L3N_MOSI_CSI_B_MISO0_2, U4.DI
- removed net FLASH_CLK: U2B2.IO_L1P_CCLK_2, U4.CLK
- removed net FLASH_CS: U2B2.IO_L65N_CSO_B_2, U4.!CS!
- removed net FLASH_MISO: R91.1, U4.DO
- removed net MCU_NSS: IC9.PA4/TIM3_CH2/SPI1_NSS/SPI3_NSS, U2B2.IO_L2P_CMPCLK_2
- removed net N$190: IC9.PA14/SWCLK, JP2.6
- removed net N$191: IC9.PA13/SWDIO, JP2.8
- removed net N$194: R92.1, U2B2.DONE_2
- removed net N$195: R93.1, U2B2.IO_L65P_INIT_B_2
- removed net N$196: R94.1, U2B2.PROGRAM_B_2
- new net FPGA_CCLK: R146.2, R91.2, U2B2.IO_L1P_CCLK_2
- new net FPGA_CSO_B: R139.2, U2B2.IO_L65N_CSO_B_2
- new net FPGA_DIN: R138.2, R147.2, U2B2.IO_L3P_D0_DIN_MISO_MISO1_2
- new net FPGA_DONE: IC9.PB9, R92.1, U2B2.DONE_2
- new net FPGA_INIT_B: IC9.PF1-OSC_OUT, R93.1, U2B2.IO_L65P_INIT_B_2
- new net FPGA_M1: R140.1, R141.2, U2B2.IO_L13P_M1_2
- new net FPGA_MOSI: R137.2, U2B2.IO_L3N_MOSI_CSI_B_MISO0_2
- new net FPGA_PROGRAM_B: IC9.PB2, R94.1, U2B2.PROGRAM_B_2
- new net MCU_FLASH_CS: IC9.PB0, R142.1
- new net MCU_FPGA_CCLK: IC9.PB15, R146.1
- new net MCU_FPGA_DIN: IC9.PB13, R147.1
- new net MCU_FPGA_NSS: IC9.PA4, U2B2.IO_L2P_CMPCLK_2
- new net N$237: R137.1, R144.2, U4.DI
- new net N$240: R138.1, R143.2, U4.DO
- new net N$241: R139.1, R142.2, U4.!CS!
- new net SWCLK: IC9.PA14, JP2.6
- new net SWDIO: IC9.PA13, JP2.8
- net +3V3: now also C228.1, IC9.VBAT, IC9.VDDA, IC9.VREF+, R141.1; no longer IC9.VDDA/VREF+
- net FPGA_RESET: now also IC9.PB7; no longer IC9.PA1/TIM2_CH2
- net GND: now also C228.2, IC9.GND, IC9.PB8-BOOT0, R140.2; no longer IC9.EP, IC9.PB8/BOOT0, IC9.VSS, IC9.VSSA, U2B2.IO_L13P_M1_2
- net MCU_AUX1: now also IC9.PA1; no longer IC9.PF0-OSC_IN
- net MCU_AUX2: now also IC9.PA2; no longer IC9.PF1-OSC_OUT
- net MCU_AUX3: now also IC9.PA3; no longer IC9.PA0/TIM2_CH1
- net MCU_FPGA_UNUSED1: now also IC9.PB5; no longer IC9.PB7/TIM4_CH2/I2C1_SDA/USART1_RX/TIM3_CH4
- net MCU_FPGA_UNUSED2: now also IC9.PB3; no longer IC9.PB3/TIM2_CH2/SPI1_SCK/SPI3_SCK/USART2_TX
- net MCU_FPGA_UNUSED3: now also IC9.PC11; no longer IC9.PA15/TIM2_CH1/TIM8_CH1/I2C1_SCL/USART2_RX/SPI1_NSS/SPI3_NSS
- net MCU_INTR: now also IC9.PB1; no longer IC9.PB0/TIM3_CH3/UCPD1_FRSTX
- net MCU_MISO: now also IC9.PA6, R143.1; no longer IC9.PA6/SPI1_MISO/TIM16_CH1/TIM3_CH1
- net MCU_MOSI: now also IC9.PA7, R144.1; no longer IC9.PA7/SPI1_MOSI/TIM17_CH1/TIM3_CH2/UCPD1_FRSTX
- net MCU_SCK: now also IC9.PA5, R145.1; no longer IC9.PA5/TIM2_CH1/SPI1_SCK/UCPD1_FRSTX
- net N$187: now also IC9.PA11; no longer IC9.PA11/TIM1_CH4/SPI2_MOSI/CAN1_RX/USB_DM
- net N$188: now also IC9.PA12; no longer IC9.PA12/TIM16_CH1/TIM4_CH2/CAN1_TX/USB_DP
- net N$192: now also IC9.PG10-NRST; no longer IC9.PG10/NRST
- net N$193: now also IC9.PC10; no longer IC9.PA2/TIM2_CH3/USART2_TX/TIM15_CH1
- net N$197: now also R145.2, R91.1, U4.CLK; no longer R91.2, U2B2.IO_L3P_D0_DIN_MISO_MISO1_2
- net N$233: now also IC9.PA9, IC9.PB6; no longer IC9.PA9/TIM1_CH2/I2C1_SCL/USART1_TX/TIM2_CH3/UCPD1_DBCC1, IC9.PB6/TIM4_CH1/TIM8_CH1/USART1_TX/UCPD1_CC1
- net N$234: now also IC9.PA10, IC9.PB4; no longer IC9.PA10/TIM1_CH3/I2C1_SDA/USART1_RX/TIM2_CH4/UCPD1_DBCC2, IC9.PB4/SPI1_MISO/SPI3_MISO/TIM16_CH1/TIM3_CH1/USART2_TX/UCPD1_CC2
- net POWER_GOOD: now also IC9.PB12; no longer IC9.PA3/TIM2_CH4/USART2_RX/TIM15_CH2
- net SCL: now also IC9.PC4; no longer IC9.PA8/I2C3_SCL/I2C2_SDA/TIM1_CH1
- net SDA: now also IC9.PA8; no longer IC9.PB5/TIM3_CH2/SPI1_MOSI/SPI3_MOSI
Other:
- note added: "Place resistors for FPGA master configuration"
- note added: "Place resistors for FPGA slave configuration"
- moved on the sheet: C167, C203, C204, C205, C206, C207, C208, C209, C210, C211, C224, C225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

Commit message: Routing + BOM
Parts:
- removed R68: 0, rcl:R-EU_R0402
- added JP1: DNP, pinhead:PINHD-2X10
- added LED10: Red, led:LEDCHIPLED_0603
- added R148: 330, rcl:R-EU_R0402
- C1, C150, C153, C2, C3, C33, C34, C35, C36, C4, C66, C67, C68: value 100n -> 100n/RF
- C121, C132: value 10n -> 100n/RF
- C131: value 10n -> 100n
- C168: value 1u/25V -> 1u
- LED1, LED5, LED6, LED7, LED8, LED9: value (none) -> Green
- LED2, LED3, LED4: value (none) -> Red
- R135, R136, R76, R88, R96: value 22 -> 20
- R137, R138, R139, R140, R91: value 0 -> DNP
- X5: value 10MHz out -> SMA_CONNECTOR
- X6: value 10MHz in -> SMA_CONNECTOR
Connections:
- net N$165 renamed TDI
- net N$173 renamed TMS
- net N$192 renamed NRST
- net N$193 renamed UART_TX
- net N$34 renamed TCK
- net N$65 renamed TDO
- removed net N$158: IC23.RF1, R68.2
- new net N$190: LED10.C, R148.1
- new net N$191: IC9.PA15, R148.2
- new net N$194: JP1.2, U2B0.IO_L34P_GCLK19_0
- new net N$195: JP1.4, U2B0.IO_L34N_GCLK18_0
- new net N$196: JP1.3, U2B0.IO_L35P_GCLK17_0
- new net N$242: JP1.6, U2B0.IO_L35N_GCLK16_0
- new net N$243: JP1.5, U2B0.IO_L36P_GCLK15_0
- new net N$244: JP1.8, U2B0.IO_L36N_GCLK14_0
- new net N$245: JP1.7, U2B0.IO_L37P_GCLK13_0
- new net N$246: JP1.10, U2B0.IO_L37N_GCLK12_0
- new net N$247: JP1.9, U2B0.IO_L62P_0
- new net N$248: JP1.12, U2B0.IO_L62N_VREF_0
- new net N$249: JP1.11, U2B0.IO_L63P_SCP7_0
- new net N$250: JP1.14, U2B0.IO_L63N_SCP6_0
- new net N$251: JP1.13, U2B0.IO_L64P_SCP5_0
- new net N$252: JP1.16, U2B0.IO_L64N_SCP4_0
- new net N$253: JP1.15, U2B0.IO_L65P_SCP3_0
- new net N$254: JP1.18, U2B0.IO_L65N_SCP2_0
- new net N$255: JP1.17, U2B0.IO_L66P_SCP1_0
- new net N$256: JP1.19, U2B0.IO_L66N_SCP0_0
- net +3V3: now also JP1.1, LED10.A
- net GND: now also JP1.20
- net N$144: now also IC23.RF1; no longer R68.1
Other:
- moved on the sheet: LED1, LED2, LED3, LED4, LED5, LED6, LED7, LED8, LED9, R105, R106, R107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

Commit message: library update
Parts:
- C1, C10, C100, C101, C102, C103, C104, C105, C107, C108, C109, C11, C110, C111, C112, C114, C115, C116, C117, C118, C119, C12, C120, C121, C122, C127, C128, C129, C13, C130, C131, C132, C133, C134, C135, C136, C137, C138, C14, C143, C144, C145, C146, C147, C148, C149, C15, C150, C151, C152, C153, C154, C155, C156, C157, C16, C167, C17, C175, C176, C178, C179, C18, C182, C183, C186, C187, C188, C19, C191, C192, C193, C194, C195, C196, C197, C198, C199, C2, C20, C200, C201, C202, C203, C204, C205, C206, C207, C208, C209, C21, C210, C211, C212, C213, C214, C215, C216, C217, C218, C219, C22, C220, C221, C222, C223, C224, C225, C226, C227, C228, C23, C24, C25, C26, C27, C28, C29, C3, C30, C31, C32, C33, C34, C35, C36, C37, C38, C39, C4, C40, C41, C42, C43, C44, C45, C46, C47, C48, C49, C5, C50, C51, C52, C53, C54, C55, C56, C57, C58, C59, C6, C60, C61, C62, C63, C64, C65, C66, C67, C68, C69, C7, C70, C71, C72, C73, C74, C75, C76, C77, C78, C79, C8, C80, C81, C82, C83, C84, C85, C86, C87, C88, C89, C9, C90, C91, C92, C93, C94, C95, C96, C97, C98, C99: device rcl:C-EUC0402 -> VNA:C-EUC0402:2
- C113, C123, C124, C139, C140, C158, C159, C160, C161, C162, C163, C164, C165, C166, C168: device VNA:C-EUC0603 -> VNA:C-EUC0603:1
- D1, D2: device diodes:D-SMB -> VNA:D-SMB
- IC1, IC37, IC5: device rf:ADL5801 -> VNA:ADL5801
- IC11, IC3, IC7: device rf:THS4521IDGKR -> VNA:THS4521IDGKR
- IC22, IC25, IC26, IC27: device rf:QPC6324 -> VNA:QPC6324
- IC23: device rf:RFSA3714 -> VNA:RFSA3714
- IC9: device custom-ic:STM32G431CB -> VNA:STM32G431CB
- J1, J2: device custom-connectors:AMPHENOL_132289 -> VNA:AMPHENOL_132289
- J4: device custom-connectors:TYPE-C16P(073) -> VNA:TYPE-C16P(073)
- JP1: device pinhead:PINHD-2X10 -> VNA:PINHD-2X10
- JP2: device pinhead:PINHD-1X10/90 -> VNA:PINHD-1X10/90
- L1, L10, L11, L12, L13, L14, L15, L16, L17, L18, L19, L2, L20, L21, L22, L23, L24, L25, L26, L27, L28, L3, L31, L32, L33, L34, L35, L36, L37, L38, L39, L4, L40, L41, L42, L43, L44, L45, L46, L47, L48, L49, L5, L50, L6, L7, L8, L9: device rf:INDUCTOR0402 -> VNA:INDUCTOR0402
- LED1, LED10, LED2, LED3, LED4, LED5, LED6, LED7, LED8, LED9: device led:LEDCHIPLED_0603 -> VNA:LEDCHIPLED_0603
- R1, R10, R100, R101, R102, R103, R104, R105, R106, R107, R108, R109, R11, R110, R111, R112, R113, R114, R115, R116, R117, R118, R119, R12, R120, R121, R122, R123, R124, R125, R126, R127, R128, R129, R13, R130, R131, R132, R133, R134, R135, R136, R137, R138, R139, R14, R140, R141, R142, R143, R144, R145, R146, R147, R148, R15, R16, R17, R18, R19, R2, R20, R21, R22, R23, R24, R25, R26, R27, R28, R29, R3, R30, R31, R32, R33, R34, R35, R36, R37, R38, R39, R4, R40, R41, R42, R43, R44, R45, R46, R47, R48, R49, R5, R50, R51, R52, R53, R54, R55, R56, R57, R58, R59, R6, R60, R61, R62, R63, R64, R65, R66, R67, R69, R7, R70, R71, R72, R73, R74, R75, R76, R77, R78, R79, R8, R80, R81, R82, R83, R84, R85, R86, R87, R88, R89, R9, R90, R91, R92, R93, R94, R95, R96, R97, R98, R99: device rcl:R-EU_R0402 -> VNA:R-EU_R0402
- T1, T2, T3: device rf:B012-617DB-1-63-B331 -> VNA:B012-617DB-1-63-B331
- TP1, TP10, TP11, TP12, TP13, TP14, TP15, TP16, TP17, TP18, TP19, TP2, TP3, TP4, TP5, TP6, TP7, TP8, TP9: device testpad:TPB1,27 -> VNA:TPB1,27
