File: Hardware/VNA.sch (EAGLE design)
At the start: 513 parts, among them IC1 ADL5801, IC10 LT5560, IC11 THS4521IDGKR, IC12 MCP33131D-10-E/MS, IC13 SI5351C, IC14 MAX2871, IC15 NCP702-3.3, IC16 RFSW6042, IC17 AP2114H, IC18 RFSW6042, IC19 MAX2871, IC2 LT5560, IC20 NCP702-3.3, IC21 AP2114H, IC22 QPC6324, IC23 RFSA3714, IC24 TRF37A73, IC25 QPC6324, IC26 QPC6324, IC27 QPC6324, IC28 LDL212PU50R, IC29 LDL212PU50R, IC3 THS4521IDGKR, IC30 LDL212PU50R, IC31 LDL212PU50R, IC32 TPS65265, IC34 NCP702-1.8, IC35 NCP702-1.8, IC36 NCP702-1.8, IC37 ADL5801, IC4 MCP33131D-10-E/MS, IC5 ADL5801, IC6 LT5560, IC7 THS4521IDGKR, IC8 MCP33131D-10-E/MS, IC9 STM32G431CB, J1 AMPHENOL_132289, J2 AMPHENOL_132289, J3 DCJ0202, J4 TYPE-C16P(073), Q1 FA-128 26MHz, T1 B012-617DB-1-63-B331, T2 B012-617DB-1-63-B331, T3 B012-617DB-1-63-B331, U2 6SLX9TQG144, U4 W25Q16BVSN, X4 DNP, X5 SMA_CONNECTOR, X6 SMA_CONNECTOR

Commit message: reworked power supply section
Parts:
- removed C223: 56p, VNA:C-EUC0402:2
- removed C224, C225, C226, C227, C228: 100n, VNA:C-EUC0402:2
- removed D2: MBRS2040LT3G, VNA:D-SMB
- removed L54: 6u8, VNA:SRN5040
- removed L55: 10u, VNA:SRN5040
- removed R143, R144, R145, R146, R147: 0, VNA:R-EU_R0402
- removed R148: 330, VNA:R-EU_R0402
- added IC33: ADL5801, VNA:ADL5801
- added L29: Ferrite, VNA:INDUCTOR0402
- added L30: 330n, VNA:INDUCTOR0402
- added R68: 620, VNA:R-EU_R0402
- C1, C2, C3: value 100n/RF -> 10u; device VNA:C-EUC0402:2 -> VNA:C-EUC1206
- C10, C11, C8: value 10n -> 10u; device VNA:C-EUC0402:2 -> VNA:C-EUC1206
- C100: value 18p -> 1u
- C101: value 56p -> 1u
- C102, C103, C118, C97: value 18p -> 100n
- C104, C105, C120, C143, C148, C157, C191, C192, C30, C39, C80: value 100n -> 10n
- C106: value 1u -> 10n; device VNA:C-EUC0603 -> VNA:C-EUC0402:2
- C107: value 10n -> DNP
- C108: value 4p -> 1u
- C109: value 4p -> 100n/RF
- C110, C71, C96: value 100n -> 100n/RF
- C111: value 56p -> 10n
- C112: value 18p -> DNP
- C113: value 4u7 -> DNP; device VNA:C-EUC0603:1 -> VNA:C-EUC0402:2
- C114, C115, C116, C122, C134, C193, C73: value 1u -> 100n
- C117, C135, C222: value 180p -> 100n
- C119: value 3n3 -> 100n
- C12, C13, C15, C49, C7: value 100n -> 10u; device VNA:C-EUC0402:2 -> VNA:C-EUC1206
- C121: value 100n/RF -> 330p
- C123, C160: value 1u -> 10n; device VNA:C-EUC0603:1 -> VNA:C-EUC0402:2
- C124: value 1u -> 120p; device VNA:C-EUC0603:1 -> VNA:C-EUC0402:2
- C125, C126: value 10u -> 330p; device VNA:C-EUC1206 -> VNA:C-EUC0402:2
- C127: value 100n -> 330p
- C128, C196: value 100n -> 150p
- C129, C131, C138, C145, C198, C203, C59: value 100n -> 1u
- C130: value 10n -> 33p
- C132, C153, C33, C4: value 100n/RF -> 100n
- C133: value 1u -> 100n/RF
- C136, C99: value 18p -> 100n/RF
- C137: value 3n3 -> 1u
- C139, C140: value 1u -> 100n; device VNA:C-EUC0603:1 -> VNA:C-EUC0402:2
- C14: value 120p -> 10u; device VNA:C-EUC0402:2 -> VNA:C-EUC1206
- C141, C142: value 10u -> 10n; device VNA:C-EUC1206 -> VNA:C-EUC0402:2
- C144, C149: value 100n -> DNP
- C146, C147, C65, C74: value 10n -> 100n/RF
- C150: value 100n/RF -> DNP
- C158, C162, C164: value 1u -> 330p; device VNA:C-EUC0603:1 -> VNA:C-EUC0402:2
- C159: value 4u7 -> 100n; device VNA:C-EUC0603:1 -> VNA:C-EUC0402:2
- C16, C17, C53: value 330p -> 10u; device VNA:C-EUC0402:2 -> VNA:C-EUC1206
- C161: value 4u7 -> 120p; device VNA:C-EUC0603:1 -> VNA:C-EUC0402:2
- C163: value 4u7 -> 330p; device VNA:C-EUC0603:1 -> VNA:C-EUC0402:2
- C165: value 1u -> 150p; device VNA:C-EUC0603:1 -> VNA:C-EUC0402:2
- C166, C168: device VNA:C-EUC0603:1 -> VNA:C-EUC0402:2
- C167, C197: value 100n -> 33p
- C169, C181, C190: value 22u -> 100n; device VNA:C-EUC1206 -> VNA:C-EUC0402:2
- C170: value 22u -> 100n/RF; device VNA:C-EUC1206 -> VNA:C-EUC0402:2
- C171, C172, C180: value 22u -> 10n; device VNA:C-EUC1206 -> VNA:C-EUC0402:2
- C173: value 10u/25V -> DNP; device VNA:C-EUC1206 -> VNA:C-EUC0402:2
- C174: value 22u -> DNP; device VNA:C-EUC1206 -> VNA:C-EUC0402:2
- C175: value 47n -> 10n
- C176: value 1n -> DNP
- C177: value 10u/25V -> 1u; device VNA:C-EUC1206 -> VNA:C-EUC0402:2
- C178: value 47n -> 100n/RF
- C179: value 8p2 -> 100n/RF
- C18: value 100n -> 1u; device VNA:C-EUC0402:2 -> VNA:C-EUC0603
- C182, C56: value 120p -> 100n
- C183, C69, C83: value DNP -> 100n
- C184, C189: value 22u -> 330p; device VNA:C-EUC1206 -> VNA:C-EUC0402:2
- C185: value 10u/25V -> 100n; device VNA:C-EUC1206 -> VNA:C-EUC0402:2
- C186: value 47n -> 100n
- C187: value 510p -> 330p
- C188: value DNP -> 330p
- C19, C27: value 330p -> 1u; device VNA:C-EUC0402:2 -> VNA:C-EUC0603:1
- C194: value 1u -> 120p
- C20, C21, C28, C79: device VNA:C-EUC0402:2 -> VNA:C-EUC0603:1
- C200, C201, C213, C214, C215, C217, C218, C219, C55, C72: value 10n -> 100n
- C202, C87: value 10n -> 1u
- C22, C23: value 100n -> 4u7; device VNA:C-EUC0402:2 -> VNA:C-EUC0603:1
- C221, C98: value 56p -> 100n
- C24, C25: value DNP -> 4u7; device VNA:C-EUC0402:2 -> VNA:C-EUC0603:1
- C26, C52, C81: value 100n -> 1u; device VNA:C-EUC0402:2 -> VNA:C-EUC0603:1
- C31: value 150p -> 4p
- C32: value 33p -> 100n
- C34: value 100n/RF -> 4p
- C35, C36, C67: value 100n/RF -> 18p
- C37: value DNP -> 18p
- C38: value 100n -> 56p
- C40, C42: value 10n -> 56p
- C41, C47: value 1u -> 56p
- C43: value 100n -> 180p
- C44, C45: value 100n -> 18p
- C46, C95: value 1u -> 18p
- C5, C51: value DNP -> 10n
- C50: value DNP -> 1u; device VNA:C-EUC0402:2 -> VNA:C-EUC0603:1
- C57: value 150p -> 100n
- C58: value 33p -> 1u
- C60: value 330p -> 1u
- C61, C62, C85, C94: value 330p -> 100n
- C63: value 1u -> 180p
- C66: value 100n/RF -> 3n3
- C78: value 1u -> 10u; device VNA:C-EUC0402:2 -> VNA:C-EUC1206
- C82: value DNP -> 10u; device VNA:C-EUC0402:2 -> VNA:C-EUC1206
- C88: value 120p -> 1u
- C89: value 150p -> 1u
- C9: value 1u -> 100p
- C90: value 33p -> 180p
- C92: value 330p -> 3n3
- C93: value 330p -> 10n
- IC1: value ADL5801 -> MIC2253; device VNA:ADL5801 -> VNA:MIC2253
- IC10: value LT5560 -> MAX2871; device VNA:LT5560 -> VNA:MAX2871
- IC11: value THS4521IDGKR -> RFSW6042; device VNA:THS4521IDGKR -> VNA:RFSW6042
- IC12: value MCP33131D-10-E/MS -> RFSW6042; device VNA:MCP33131D-10-E/MS -> VNA:RFSW6042
- IC13: value SI5351C -> QPC6324; device VNA:SI5351C -> VNA:QPC6324
- IC14: value MAX2871 -> RFSA3714; device VNA:MAX2871 -> VNA:RFSA3714
- IC15: value NCP702-3.3 -> TRF37A73; device VNA:NCP702 -> VNA:TRF37A73
- IC16, IC18: value RFSW6042 -> QPC6324; device VNA:RFSW6042 -> VNA:QPC6324
- IC17: value AP2114H -> QPC6324; device VNA:AP2114H -> VNA:QPC6324
- IC19: value MAX2871 -> AP2114H; device VNA:MAX2871 -> VNA:AP2114H
- IC2: value LT5560 -> LM3370SD-4221; device VNA:LT5560 -> VNA:LM3370
- IC21: value AP2114H -> MAX2871; device VNA:AP2114H -> VNA:MAX2871
- IC22, IC27: value QPC6324 -> LT5560; device VNA:QPC6324 -> VNA:LT5560
- IC23: value RFSA3714 -> THS4521IDGKR; device VNA:RFSA3714 -> VNA:THS4521IDGKR
- IC24: value TRF37A73 -> ADL5801; device VNA:TRF37A73 -> VNA:ADL5801
- IC25: value QPC6324 -> NCP702-1.8; device VNA:QPC6324 -> VNA:NCP702
- IC26: value QPC6324 -> MCP33131D-10-E/MS; device VNA:QPC6324 -> VNA:MCP33131D-10-E/MS
- IC28: value LDL212PU50R -> THS4521IDGKR; device VNA:LDL212PU50R -> VNA:THS4521IDGKR
- IC29: value LDL212PU50R -> ADL5801; device VNA:LDL212PU50R -> VNA:ADL5801
- IC3: value THS4521IDGKR -> LDL212PU50R; device VNA:THS4521IDGKR -> VNA:LDL212PU50R
- IC30: value LDL212PU50R -> NCP702-1.8; device VNA:LDL212PU50R -> VNA:NCP702
- IC31: value LDL212PU50R -> MCP33131D-10-E/MS; device VNA:LDL212PU50R -> VNA:MCP33131D-10-E/MS
- IC32: value TPS65265 -> THS4521IDGKR; device VNA:TPS65265 -> VNA:THS4521IDGKR
- IC35: value NCP702-1.8 -> MCP33131D-10-E/MS; device VNA:NCP702 -> VNA:MCP33131D-10-E/MS
- IC36: value NCP702-1.8 -> LT5560; device VNA:NCP702 -> VNA:LT5560
- IC37: value ADL5801 -> STM32G431CB; device VNA:ADL5801 -> VNA:STM32G431CB
- IC4: value MCP33131D-10-E/MS -> LDL212PU50R; device VNA:MCP33131D-10-E/MS -> VNA:LDL212PU50R
- IC5: value ADL5801 -> LDL212PU50R; device VNA:ADL5801 -> VNA:LDL212PU50R
- IC6: value LT5560 -> LDL212PU50R; device VNA:LT5560 -> VNA:LDL212PU50R
- IC7: value THS4521IDGKR -> SI5351C; device VNA:THS4521IDGKR -> VNA:SI5351C
- IC8: value MCP33131D-10-E/MS -> AP2114H; device VNA:MCP33131D-10-E/MS -> VNA:AP2114H
- IC9: value STM32G431CB -> NCP702-3.3; device VNA:STM32G431CB -> VNA:NCP702
- J1: value AMPHENOL_132289 -> DNP; device VNA:AMPHENOL_132289 -> VNA:DCJ0202
- J3: value DCJ0202 -> AMPHENOL_132289; device VNA:DCJ0202 -> VNA:AMPHENOL_132289
- JP1: device VNA:PINHD-2X10 -> VNA:PINHD-1X10/90
- JP2: device VNA:PINHD-1X10/90 -> VNA:PINHD-2X10
- L1, L2, L3: value 330n -> 2u2; device VNA:INDUCTOR0402 -> VNA:SRN5040
- L10, L25, L26, L9: value 33n -> Ferrite
- L11, L12, L17: value 330n -> 120n
- L13: value 68n -> 120n
- L14, L24: value 68n -> 330n
- L15, L16: value 33n -> 120n
- L19, L20, L21, L22, L27, L28, L6: value 330n -> Ferrite
- L23, L7, L8: value 68n -> Ferrite
- L31, L38, L39, L40, L41, L46, L47: value Ferrite -> 330n
- L32, L33: value 120n -> 330n
- L34, L35: value 120n -> 68n
- L36, L37: value 120n -> 33n
- L4, L5: value Ferrite -> 2u2; device VNA:INDUCTOR0402 -> VNA:SRN5040
- L42, L43, L48, L49: value Ferrite -> 68n
- L44: value 330n -> 33n
- L45, L50: value Ferrite -> 33n
- L51: value 10u -> 33n; device VNA:SRN5040 -> VNA:INDUCTOR0402
- L52, L53: value 6u8 -> 330n; device VNA:SRN5040 -> VNA:INDUCTOR0402
- LED1, LED5: value Green -> Red
- LED10, LED2: value Red -> Green
- LP2: value LP0603A1880ANTR -> LP0603N3500ANTR
- LP3: value LP0603N3500ANTR -> LP0603A1880ANTR
- R10: value 620 -> 5k1
- R100, R111, R112, R113: value 10k -> DNP
- R101: value 10k -> 1k
- R102, R103, R80, R86, R97, R98, R99: value 10k -> 220
- R104, R49: value 10k -> 0
- R105, R106, R107, R108, R109, R110: value 330 -> 0
- R11, R25: value 1k -> 10k
- R116, R127, R128, R130, R131: value DNP -> 10k
- R117, R121, R122, R19, R20, R31: value 220 -> 10k
- R118, R119: value 220 -> 20
- R12: value 18 -> 49R9
- R120: value 220 -> 330
- R123, R126, R91: value DNP -> 20
- R124: value 0 -> 20
- R125, R77: value DNP -> 0
- R129: value 0 -> 10k
- R13: value 620 -> 49R9
- R134: value 10k -> 330
- R135, R136, R39: value 20 -> 330
- R137, R138, R139, R140: value DNP -> 330
- R14: value 330 -> 49R9
- R141, R142: value 0 -> 330
- R15: value 200 -> 1k8
- R16: value 200 -> 82
- R17: value 6k8 -> 330
- R18: value 6k8 -> 10k
- R2: value 620 -> 4k7
- R21, R5: value 620 -> 10k
- R22, R23, R24, R6: value 49R9 -> 10k
- R26: value 330 -> 2R7
- R27: value 200 -> 406
- R28: value 200 -> 56
- R29: value 6k8 -> 2R7
- R3: value 18 -> 10k
- R30: value 6k8 -> 5k1
- R32: value 220 -> 49R9
- R33, R72: value 56 -> 49R9
- R34, R35, R38, R76: value 20 -> 49R9
- R36: value 56 -> 1k8
- R37: value 56 -> 82
- R4: value 620 -> 38k3
- R40: value 56 -> 620
- R41: value 1k -> 620
- R42: value 330 -> 18
- R43, R44: value 200 -> 620
- R45, R46: value 4k7 -> 49R9
- R47, R48: value 220 -> DNP
- R50: value 1k8 -> 49R9
- R51: value 82 -> DNP
- R52: value 330 -> DNP
- R53, R61: value 5k1 -> 220
- R54, R62: value 49R9 -> 220
- R55: value 49R9 -> 6k8
- R56, R83: value 10k -> 6k8
- R57: value 49R9 -> DNP
- R58: value 1k8 -> 220
- R59: value 82 -> 220
- R60: value 330 -> 1k
- R63, R66: value 49R9 -> 56
- R64, R92: value 10k -> 20
- R65: value 49R9 -> 20
- R67: value 49R9 -> 620
- R69: value 2R7 -> 18
- R7: value 49R9 -> 100
- R70: value 2R7 -> 620
- R71: value 406 -> 620
- R73: value 100 -> 49R9
- R74: value 62 -> DNP
- R75: value 100 -> DNP
- R78: value 51k -> DNP
- R79: value 82k -> DNP
- R8: value 49R9 -> 62
- R81: value 91k -> 220
- R82: value 16k -> 6k8
- R84: value 20k -> DNP
- R85: value 30k -> 220
- R87: value 45k3 -> 1k
- R88, R96: value 20 -> 220
- R89: value DNP -> 220
- R9: value 620 -> 100
- R90, R93: value 10k -> 56
- R94, R95: value 10k -> 4k7
- renumbered U4 to U1, X4 to X3, X5 to X2, X6 to X1
Connections:
- removed net +12V: C173.1, C177.1, C185.1, D1.C, D2.C, IC32G1.VIN, IC32G2.VIN, IC32G3.VIN
- removed net N$167: IC32COMMON.PSM, R77.2
- removed net N$168: C178.2, IC32G1.BST
- removed net N$169: C178.1, IC32G1.LX, L52.1
- removed net N$170: C175.2, IC32G2.BST
- removed net N$172: IC32G2.COMP, R82.2
- removed net N$174: IC32G1.COMP, R79.2
- removed net N$176: C183.2, IC32G1.FB, R80.2, R81.1
- removed net N$178: C179.2, IC32G2.FB, R83.2, R84.1
- removed net N$180: C186.2, IC32G3.BST
- removed net N$182: IC32G3.COMP, R85.2
- removed net N$184: C188.2, IC32G3.FB, R86.2, R87.1
- removed net N$226: C187.2, R85.1
- removed net N$227: C176.2, R82.1
- removed net N$232: D1.A, J3.1
- removed net POWER_GOOD: IC32COMMON.PGOOD, IC9.PB12
- removed net SWITCHING_SYNC: IC32COMMON.ROSC, R78.2
- new net +5V: C1.1, C2.1, C3.1, C6.2, IC1.VIN, IC2BUCK1.EN, IC2BUCK1.VIN, IC2BUCK2.EN, IC2BUCK2.VIN, IC2CONTROL.VDD, J1.1, L1.1, R125.2
- new net EN_6V: IC1.EN, IC37.PB12
- new net N$158: C9.2, IC1.FB, R4.1, R5.2
- new net N$165: C4.2, IC1.SS
- new net N$34: D1.A, IC1.SW, L1.2
- new net N$65: IC1.COMP, R1.2
- net +3V3: now also C132.2, C14.1, C15.1, C169.2, C201.2, C208.1, C209.1, C210.1, C212.1, C214.1, C216.1, C218.1, C220.1, C221.1, C222.1, C54.1, C55.1, C83.1, C84.1, IC10.VCC_DIG, IC10.VDD_SD, IC21.VCC_DIG, IC21.VDD_SD, IC26.DVIO, IC26.SDI, IC31.DVIO, IC31.SDI, IC35.DVIO, IC35.SDI, IC37.VBAT, IC37.VDD, IC37.VDDA, IC37.VREF+, IC7.VDD, JP1.5, JP2.1, L10.1, L21.1, L22.1, L23.1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; no longer C110.2, C120.1, C127.1, C138.1, C143.1, C189.1, C190.1, C191.1, C192.1, C203.1, C204.1, C205.1, C224.1, C225.1, C226.1, C227.1, C228.1, C64.2, C96.2, IC12.DVIO, IC12.SDI, IC13.VDD, IC14.VCC_DIG, IC14.VDD_SD, IC19.VCC_DIG, IC19.VDD_SD, IC4.DVIO, IC4.SDI, IC8.DVIO, IC8.SDI, IC9.VBAT, IC9.VDD, IC9.VDDA, IC9.VREF+, JP1.1, JP2.5, L31.1, L4.1, L42.1, L43.1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
- net +5V/1: now also C102.2, C103.2, C104.1, C105.1, C106.1, C108.1, C111.1, C115.2, C119.1, C122.1, C129.1, C26.2, IC22.VCC, IC23.V+, IC24.VPDT, IC24.VPLO, IC24.VPRF, IC25.EN, IC25.VIN, IC26.VREF, L32.1, L33.1, L6.2, R53.1, R54.1, R60.1, TP5.TP; no longer C12.1, C13.1, C164.2, C193.1, C200.1, C201.1, C202.1, C22.2, C23.2, C30.2, C8.1, C9.1, IC2.VCC, IC3.V+, IC34.EN, IC34.VIN, IC37.VPDT, IC37.VPLO, IC37.VPRF, IC4.VREF, L1.1, L2.1, L47.2, R11.1, R15.1, R16.1, TP7.TP
- net +5V/2: now also C139.2, C140.2, C141.1, C142.1, C143.1, C145.1, C148.1, C152.2, C156.1, C159.1, C166.1, C27.2, IC27.VCC, IC28.V+, IC29.VPDT, IC29.VPLO, IC29.VPRF, IC30.EN, IC30.VIN, IC31.VREF, L40.1, L41.1, L7.2, R80.1, R81.1, R87.1, TP7.TP; no longer C165.2, C213.1, C214.1, C215.1, C28.1, C40.1, C41.1, C43.1, C44.1, C48.2, C49.2, C54.2, IC1.VPDT, IC1.VPLO, IC1.VPRF, IC35.EN, IC35.VIN, IC6.VCC, IC7.V+, IC8.VREF, L12.1, L48.2, L6.1, R25.1, R27.1, R28.1, TP9.TP
- net +5V/3: now also C171.1, C172.1, C175.1, C177.1, C180.1, C181.2, C190.1, C193.1, C195.1, C204.2, C205.2, C28.2, IC32.V+, IC33.VPDT, IC33.VPLO, IC33.VPRF, IC34.EN, IC34.VIN, IC35.VREF, IC36.VCC, L46.1, L47.1, L8.2, R101.1, R102.1, R103.1, TP9.TP; no longer C166.2, C217.1, C218.1, C219.1, C72.1, C73.1, C75.1, C76.1, C80.2, C81.2, C86.2, C95.1, IC10.VCC, IC11.V+, IC12.VREF, IC36.EN, IC36.VIN, IC5.VPDT, IC5.VPLO, IC5.VPRF, L21.1, L22.1, L49.2, R41.1, R43.1, R44.1, TP11.TP
- net +5V/4: now also C49.1, C50.1, C78.1, C79.1, IC19.VIN, IC8.VIN, IC9.EN, IC9.VIN, L9.2, TP11.TP; no longer C123.1, C125.1, C139.1, C141.1, IC15.EN, IC15.VIN, IC17.VIN, IC21.VIN, L50.2, TP13.TP
- net AMP_PWDN: now also IC15.PWDN; no longer IC24.PWDN
- net ATT_D0: now also IC14.D0; no longer IC23.D0
- net ATT_D1: now also IC14.D1; no longer IC23.D1
- net ATT_D2: now also IC14.D2; no longer IC23.D2
- net ATT_D3: now also IC14.D3; no longer IC23.D3
- net ATT_D4: now also IC14.D4; no longer IC23.D4
- net ATT_D5: now also IC14.D5; no longer IC23.D5
- net ATT_D6: now also IC14.D6; no longer IC23.D6
- net FILT_IN_C1: now also R21.2; no longer R99.2
- net FILT_IN_C2: now also R20.2; no longer R100.2
- net FILT_OUT_C1: now also R24.2; no longer R104.2
- net FILT_OUT_C2: now also R22.2; no longer R103.2
- net FPGA_CCLK: now also R109.2, R111.2; no longer R146.2, R91.2
- net FPGA_CLK: now also IC7.CLK7, R126.1; no longer IC13.CLK7, R96.1
- net FPGA_CSO_B: now also R114.2; no longer R139.2
- net FPGA_DIN: now also R110.2, R113.2; no longer R138.2, R147.2
- net FPGA_DONE: now also IC37.PB9, R129.1; no longer IC9.PB9, R92.1
- net FPGA_INIT_B: now also IC37.PF1-OSC_OUT, R128.1; no longer IC9.PF1-OSC_OUT, R93.1
- net FPGA_M1: now also R108.2, R115.1; no longer R140.1, R141.2
- net FPGA_MOSI: now also R112.2; no longer R137.2
- net FPGA_PROGRAM_B: now also IC37.PB2, R127.1; no longer IC9.PB2, R94.1
- net FPGA_RESET: now also IC37.PB7; no longer IC9.PB7
- net GND: now also C1.2, C10.2, C102.1, C103.1, C104.2, C105.2, C106.2, C108.2, C11.2, C115.1, C119.2, C125.1, C131.2, C132.1, C134.1, C139.1, C14.2, C140.1, C15.2, C152.1, C153.2, C155.1, C159.2, C16.2, C164.2, C166.2, C168.2, C169.1, C17.2, C175.2, C181.1, C182.2, C186.1, C19.1, C199.1, C2.2, C20.1, C201.1, C204.1, C205.1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; no longer C100.2, C101.2, C102.2, C103.2, C104.1, C105.1, C106.1, C108.1, C109.1, C110.1, C112.2, C113.1, C114.2, C115.2, C120.2, C123.2, C124.2, C125.2, C126.2, C128.2, C133.2, C134.2, C135.2, C136.1, C138.2, C139.2, C140.2, C144.2, C149.2, C151.2, C152.2, C155.2, C158.1, C159.1, C160.1, C161.1, C163.1, C164.1, C165.1, C166.1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
- net HIGHBAND_SELECT: now also IC13.CTL1; no longer IC22.CTL1
- net LO1_CE: now also IC21.CE, R31.2; no longer IC19.CE, R64.2
- net LO1_CLK: now also IC21.CLK; no longer IC19.CLK
- net LO1_LD: now also IC21.LD; no longer IC19.LD
- net LO1_LE: now also IC21.LE; no longer IC19.LE
- net LO1_MOSI: now also IC21.DATA; no longer IC19.DATA
- net LO1_MUX: now also IC21.MUX; no longer IC19.MUX
- net LO1_REF: now also C80.1, IC7.CLK5; no longer C146.1, IC13.CLK5
- net LO1_RF_EN: now also IC21.RFOUT_EN; no longer IC19.RFOUT_EN
- net LOWBAND_SELECT: now also IC13.CTL2; no longer IC22.CTL2
- net MCU_AUX1: now also IC37.PA1; no longer IC9.PA1
- net MCU_AUX2: now also IC37.PA2; no longer IC9.PA2
- net MCU_AUX3: now also IC37.PA3; no longer IC9.PA3
- net MCU_FLASH_CS: now also IC37.PB0, R107.1; no longer IC9.PB0, R142.1
- net MCU_FPGA_CCLK: now also IC37.PB15, R109.1; no longer IC9.PB15, R146.1
- net MCU_FPGA_DIN: now also IC37.PB13, R110.1; no longer IC9.PB13, R147.1
- net MCU_FPGA_NSS: now also IC37.PA4; no longer IC9.PA4
- net MCU_FPGA_UNUSED1: now also IC37.PB5; no longer IC9.PB5
- net MCU_FPGA_UNUSED2: now also IC37.PB3; no longer IC9.PB3
- net MCU_FPGA_UNUSED3: now also IC37.PC11; no longer IC9.PC11
- net MCU_INTR: now also IC37.PB1; no longer IC9.PB1
- net MCU_MISO: now also IC37.PA6, R106.1; no longer IC9.PA6, R143.1
- net MCU_MOSI: now also IC37.PA7, R105.1; no longer IC9.PA7, R144.1
- net MCU_SCK: now also IC37.PA5, R104.1; no longer IC9.PA5, R145.1
- net N$1: now also C96.2, R40.1, R41.2, R42.2; no longer C2.2, R1.2, R2.1, R3.2
- net N$10: now also C107.2, C109.1; no longer C3.1, C5.2
- net N$100: now also C22.2, IC3.SENSE, IC3.VOUT, L6.1; no longer C113.2, IC28.SENSE, IC28.VOUT, L47.1
- net N$101: now also C35.1, IC7.CLK4, L11.1; no longer C99.1, IC13.CLK4, L33.1
- net N$102: now also C60.1, IC10.BIAS_FILT; no longer C116.1, IC14.BIAS_FILT
- net N$103: now also C39.1, IC7.CLK6; no longer C65.1, IC13.CLK6
- net N$104: now also C66.2, R16.1; no longer C119.2, R51.1
- net N$105: now also IC10.SW, R16.2, R17.1; no longer IC14.SW, R51.2, R52.1
- net N$106: now also IC10.RSET, R10.2; no longer IC14.RSET, R53.2
- net N$107: now also C30.1; no longer C107.1
- net N$108: now also C30.2, IC7.CLKIN; no longer C107.2, IC13.CLKIN
- net N$109: now also C32.2, C33.2, IC7.VDDOA, IC7.VDDOB, IC7.VDDOC, IC7.VDDOD, L10.2; no longer C104.2, C105.2, IC13.VDDOA, IC13.VDDOB, IC13.VDDOC, IC13.VDDOD, L31.2
- net N$11: now also C117.1, IC24.LO-; no longer C6.1, IC37.LO-
- net N$110: now also C56.1, C61.1, C64.1, IC10.VCC_RF, IC10.VCC_VCO, L19.2, R12.2, R13.2, TP14.TP; no longer C129.1, C196.1, C197.1, IC14.VCC_RF, IC14.VCC_VCO, L38.2, R54.2, R55.2, TP16.TP
- net N$111: now also C86.1, IC21.VCC_CP, IC21.VCC_PLL, L29.2, TP15.TP; no longer C144.1, IC19.VCC_CP, IC19.VCC_PLL, L41.2, TP18.TP
- net N$112: now also IC7.OEB, R6.2; no longer IC13.OEB, R49.2
- net N$113: now also C34.2, IC7.XA; no longer C109.2, IC13.XA
- net N$114: now also C31.2, IC7.XB; no longer C108.2, IC13.XB
- net N$115: now also C95.2, IC21.TUNE, R36.2; no longer C136.2, IC19.TUNE, R58.2
- net N$116: now also C51.2, IC10.REF_IN; no longer C130.2, IC14.REF_IN
- net N$117: now also C65.1, IC10.RFOUTA_P, R12.1; no longer C132.1, IC14.RFOUTA_P, R55.1
- net N$118: now also C62.2, IC10.RFOUTA_N, R13.1; no longer C131.2, IC14.RFOUTA_N, R54.1
- net N$119: now also C62.1, R14.2; no longer C131.1, R57.2
- net N$12: now also C114.2, IC24.LO+; no longer C7.2, IC37.LO+
- net N$120: now also C65.2, IC11.ANT; no longer C132.2, IC16.ANT
- net N$121: now also IC11.RF1, IC12.RF3; no longer IC16.RF1, IC18.RF3
- net N$122: now also IC11.RF2; no longer IC16.RF2
- net N$123: now also IC12.RF4; no longer IC18.RF4
- net N$124: now also IC12.RF2, LP2.OUT; no longer IC18.RF2, LP3.OUT
- net N$125: now also IC12.RF1, LP3.OUT; no longer IC18.RF1, LP2.OUT
- net N$126: now also IC11.RF3, LP3.IN; no longer IC16.RF3, LP2.IN
- net N$127: now also IC11.RF4, LP2.IN; no longer IC16.RF4, LP3.IN
- net N$128: now also C53.1, IC8.VOUT, L19.1; no longer C126.1, IC17.VOUT, L38.1
- net N$129: now also C52.1, IC9.VOUT, L20.1; no longer C124.1, IC15.VOUT, L39.1
- net N$13: now also C125.2, C126.1, IC26.AIN+, R61.1; no longer C16.1, C17.2, IC4.AIN+, R117.1
- net N$130: now also C68.1, IC12.ANT; no longer C121.1, IC18.ANT
- net N$131: now also C90.1, C92.1, IC21.CP_OUT, R36.1; no longer C135.1, C137.1, IC19.CP_OUT, R58.1
- net N$132: now also C87.1, IC21.REG; no longer C122.1, IC19.REG
- net N$133: now also C88.1, IC21.NOISE_FILT; no longer C133.1, IC19.NOISE_FILT
- net N$134: now also C89.1, IC21.BIAS_FILT; no longer C134.1, IC19.BIAS_FILT
- net N$135: now also C92.2, R37.1; no longer C137.2, R59.1
- net N$136: now also IC21.SW, R37.2, R39.1; no longer IC19.SW, R59.2, R60.1
- net N$137: now also IC21.RSET, R30.2; no longer IC19.RSET, R61.2
- net N$138: now also C85.1, C91.1, C94.1, IC21.VCC_RF, IC21.VCC_VCO, L28.2, R32.2, R33.2, R34.2, R35.2, TP16.TP; no longer C145.1, C198.1, C199.1, IC19.VCC_RF, IC19.VCC_VCO, L40.2, R62.2, R63.2, R65.2, R66.2, TP19.TP
- net N$139: now also C80.2, IC21.REF_IN; no longer C146.2, IC19.REF_IN
- net N$14: now also C120.1, IC24.OUT+, L32.2; no longer C11.1, IC37.OUT+, L1.2
- net N$140: now also C69.1, IC13.VCC, L21.2; no longer C149.1, IC22.VCC, L42.2
- net N$141: now also C93.1, R38.2; no longer C147.1, R67.2
- net N$142: now also C82.1, IC19.VOUT, L28.1; no longer C142.1, IC21.VOUT, L40.1
- net N$143: now also C81.1, L29.1; no longer C140.1, L41.1
- net N$144: now also IC13.RF_COM, IC14.RF1; no longer IC22.RF_COM, IC23.RF1
- net N$145: now also C70.1, IC14.LE, IC14.VDD, L22.2; no longer C148.1, IC23.LE, IC23.VDD, L43.2
- net N$146: now also C71.1, IC14.RF2; no longer C150.1, IC23.RF2
- net N$147: now also C93.2, IC21.RFOUTB_N, R35.1; no longer C147.2, IC19.RFOUTB_N, R66.1
- net N$148: now also C71.2, IC15.RFIN; no longer C150.2, IC24.RFIN
- net N$149: now also C74.1, IC15.RFOUT, L24.2; no longer C153.1, IC24.RFOUT, L44.2
- net N$15: now also C123.1, IC24.OUT-, L33.2; no longer C10.1, IC37.OUT-, L2.2
- net N$150: now also C74.2, R26.1; no longer C153.2, R69.1
- net N$151: now also IC16.RF_COM, R29.2; no longer IC25.RF_COM, R70.2
- net N$152: now also C72.1, C73.1, IC15.VCC, L23.2, L24.1; no longer C151.1, C152.1, IC24.VCC, L44.1, L45.2
- net N$153: now also R26.2, R27.2, R29.1; no longer R69.2, R70.1, R71.2
- net N$154: now also IC16.RF2, IC18.RF_COM; no longer IC25.RF2, IC26.RF_COM
- net N$155: now also IC16.RF1, IC17.RF1; no longer IC25.RF1, IC27.RF1
- net N$156: now also C76.1, IC18.VCC, L27.2; no longer C156.1, IC26.VCC, L46.2
- net N$157: now also C38.1, IC7.CLK0, L14.1; no longer C223.1, IC13.CLK0, L20.1
- net N$159: now also C48.2, R8.2, R9.2; no longer C157.2, R74.2, R75.2
- net N$16: now also C123.2, C124.2, L35.1; no longer C10.2, C14.2, L8.1
- net N$160: now also C37.1, IC7.CLK2, L13.1; no longer C112.1, IC13.CLK2, L37.1
- net N$161: now also C23.2, IC4.SENSE, IC4.VOUT, L7.1; no longer C159.2, IC29.SENSE, IC29.VOUT, L48.1
- net N$162: now also IC1.OVP, R2.1, R3.2; no longer C168.2, IC32COMMON.V7V
- net N$163: now also C16.1, C17.1, C18.2, C19.2, C20.2, C21.2, IC3.EN, IC3.VIN, IC4.EN, IC4.VIN, IC5.EN, IC5.VIN, IC6.EN, IC6.VIN, L5.2, TP3.TP; no longer C106.2, C158.2, C160.2, C162.2, C174.1, C181.1, IC28.EN, IC28.VIN, IC29.EN, IC29.VIN, IC30.EN, IC30.VIN, IC31.EN, IC31.VIN, L51.2, TP5.TP
- net N$164: now also C24.2, IC5.SENSE, IC5.VOUT, L8.1; no longer C161.2, IC30.SENSE, IC30.VOUT, L49.1
- net N$166: now also C25.2, IC6.SENSE, IC6.VOUT, L9.1; no longer C163.2, IC31.SENSE, IC31.VOUT, L50.1
- net N$17: now also C128.2, L35.2, L37.1; no longer C31.2, L10.1, L8.2
- net N$171: now also IC2BUCK1.SW, L2.1; no longer C175.1, IC32G2.LX, L53.1
- net N$175: now also R135.2; no longer R109.2
- net N$177: now also C12.1, C13.1, C9.1, D1.C, L5.1, R2.2, R4.2; no longer C170.1, C171.1, C183.1, L51.1, L52.2, R81.2
- net N$179: now also R136.2; no longer R108.2
- net N$18: now also C98.2, IC22.LO+; no longer C15.2, IC2.LO+
- net N$181: now also IC2BUCK2.SW, L3.1; no longer C186.1, IC32G3.LX, L54.1
- net N$183: now also C11.1, C8.1, IC2BUCK2.FB, L3.2, L4.1; no longer C180.1, C184.1, C188.1, L54.2, L55.1, R87.2
- net N$185: now also R125.1; no longer D2.A
- net N$186: now also R119.2; no longer R76.2
- net N$187: now also IC37.PA11, R118.2; no longer IC9.PA11, R88.2
- net N$188: now also IC37.PA12, R119.1; no longer IC9.PA12, R76.1
- net N$189: now also R118.1; no longer R88.1
- net N$19: now also C118.2, IC24.VSET, R57.1, R60.2; no longer C212.2, IC37.VSET, R11.2, R114.1
- net N$190: now also LED1.C, R120.1; no longer LED10.C, R148.1
- net N$191: now also IC37.PA15, R120.2; no longer IC9.PA15, R148.2
- net N$194: now also JP2.2; no longer JP1.2
- net N$195: now also JP2.4; no longer JP1.4
- net N$196: now also JP2.3; no longer JP1.3
- net N$197: now also R104.2, R111.1; no longer R145.2, R91.1
- net N$198: now also R126.2; no longer R96.2
- net N$199: now also IC11.C1, R18.1, R21.1; no longer IC16.C1, R97.1, R99.1
- net N$2: now also R42.1, R43.2, R44.1, R45.2, R46.2; no longer R3.1, R4.2, R5.1, R6.2, R7.2
- net N$20: now also C126.2, C127.1, IC26.AIN-, R62.1; no longer C16.2, C19.1, IC4.AIN-, R118.1
- net N$200: now also IC11.C2, R19.1, R20.1; no longer IC16.C2, R100.1, R98.1
- net N$201: now also IC12.C2, R22.1, R23.1; no longer IC18.C2, R101.1, R103.1
- net N$202: now also IC12.C1, R24.1, R25.1; no longer IC18.C1, R102.1, R104.1
- net N$203: now also C131.1, IC25.VOUT, IC26.AVDD, TP17.TP; no longer C194.1, IC34.VOUT, IC4.AVDD, TP2.TP
- net N$204: now also C168.1, IC30.VOUT, IC31.AVDD, TP18.TP; no longer C63.1, IC35.VOUT, IC8.AVDD, TP4.TP
- net N$205: now also C198.1, IC34.VOUT, IC35.AVDD, TP19.TP; no longer C195.1, IC12.AVDD, IC36.VOUT, TP15.TP
- net N$206: now also LED10.C, R142.1; no longer LED9.C, R14.1
- net N$207: now also LED9.C, R141.1; no longer LED8.C, R26.1
- net N$208: now also LED8.C, R140.1; no longer LED7.C, R42.1
- net N$209: now also LED7.C, R139.1; no longer LED6.C, R105.1
- net N$21: now also C133.2, R67.1, R68.2, R69.2; no longer C34.2, R10.1, R12.2, R9.2
- net N$210: now also LED6.C, R138.1; no longer LED5.C, R106.1
- net N$211: now also LED5.C, R137.1; no longer LED4.C, R107.1
- net N$212: now also LED4.C, R136.1; no longer LED3.C, R108.1
- net N$213: now also LED3.C, R135.1; no longer LED2.C, R109.1
- net N$214: now also LED2.C, R134.1; no longer LED1.C, R110.1
- net N$215: now also R142.2; no longer R14.2
- net N$216: now also R141.2; no longer R26.2
- net N$217: now also IC22.IN-, L31.1, R64.1, R66.1; no longer IC2.IN-, L11.1, R34.1, R36.1
- net N$218: now also IC22.IN+, L30.1, R65.1, R66.2; no longer IC2.IN+, L3.1, R35.1, R36.2
- net N$219: now also R140.2; no longer R42.2
- net N$22: now also R69.1, R70.2, R71.1, R72.2, R73.2; no longer R12.1, R13.2, R21.1, R22.2, R23.2
- net N$220: now also R139.2; no longer R105.2
- net N$221: now also R138.2; no longer R106.2
- net N$222: now also R137.2; no longer R107.2
- net N$223: now also IC27.IN-, L39.1, R91.1, R93.1; no longer IC6.IN-, L18.1, R38.1, R40.1
- net N$224: now also R124.2; no longer R135.2
- net N$225: now also C5.2, R1.1; no longer C182.2, R79.1
- net N$228: now also R123.2; no longer R136.2
- net N$229: now also IC24.DETO, R57.2; no longer IC37.DETO, R114.2
- net N$23: now also IC27.IN+, L38.1, R92.1, R93.2; no longer IC6.IN+, L17.1, R39.1, R40.2
- net N$230: now also IC29.DETO, R84.2; no longer IC1.DETO, R115.2
- net N$231: now also IC33.DETO, R100.2; no longer IC5.DETO, R116.2
- net N$233: now also IC37.PA9, IC37.PB6; no longer IC9.PA9, IC9.PB6
- net N$234: now also IC37.PA10, IC37.PB4; no longer IC9.PA10, IC9.PB4
- net N$235: now also C75.1, IC16.VCC, L25.1; no longer C155.1, IC25.VCC, L5.1
- net N$236: now also C99.2, R47.2, R49.1, R51.1; no longer C1.2, R124.1, R125.2, R126.1
- net N$237: now also R105.2, R112.1; no longer R137.1, R144.2
- net N$238: now also C136.2, R74.2, R77.1, R78.1; no longer C33.2, R129.1, R130.2, R131.1
- net N$239: now also C136.1, J3.1; no longer C33.1, J2.1
- net N$24: now also C97.2, IC22.LO-; no longer C18.2, IC2.LO-
- net N$240: now also R106.2, R113.1; no longer R138.1, R143.2
- net N$241: now also R107.2, R114.1; no longer R139.1, R142.2
- net N$242: now also JP2.6; no longer JP1.6
- net N$243: now also JP2.5; no longer JP1.5
- net N$244: now also JP2.8; no longer JP1.8
- net N$245: now also JP2.7; no longer JP1.7
- net N$246: now also JP2.10; no longer JP1.10
- net N$247: now also JP2.9; no longer JP1.9
- net N$248: now also JP2.12; no longer JP1.12
- net N$249: now also JP2.11; no longer JP1.11
- net N$25: now also R72.1, R75.1, R77.2, R79.2; no longer R127.2, R128.1, R129.2, R22.1
- net N$250: now also JP2.14; no longer JP1.14
- net N$251: now also JP2.13; no longer JP1.13
- net N$252: now also JP2.16; no longer JP1.16
- net N$253: now also JP2.15; no longer JP1.15
- net N$254: now also JP2.18; no longer JP1.18
- net N$255: now also JP2.17; no longer JP1.17
- net N$256: now also JP2.19; no longer JP1.19
- net N$26: now also R73.1, R76.1; no longer R23.1, R24.1
- net N$27: now also C100.1, IC22.OUT+, R53.2; no longer C20.1, IC2.OUT+, R15.2
- net N$28: now also C101.1, IC22.OUT-, R54.2; no longer C21.1, IC2.OUT-, R16.2
- net N$29: now also C146.2, IC29.IN+; no longer C35.2, IC1.IN+
- net N$3: now also C120.2, C124.1, L34.1; no longer C11.2, C14.1, L7.1
- net N$30: now also C147.2, IC29.IN-; no longer C36.2, IC1.IN-
- net N$31: now also C113.1, IC23.+OUT, R56.1, R59.2; no longer C25.1, IC3.+OUT, R18.1, R19.2
- net N$32: now also C112.2, IC23.-OUT, R55.2, R58.2; no longer C24.2, IC3.-OUT, R17.2, R20.2
- net N$33: now also C128.1, L34.2, L36.1; no longer C31.1, L7.2, L9.1
- net N$35: now also C144.1, C147.1; no longer C36.1, C37.1
- net N$36: now also C144.2, C146.1; no longer C35.1, C37.2
- net N$37: now also C154.1, IC29.LO-; no longer C38.1, IC1.LO-
- net N$38: now also C151.2, IC29.LO+; no longer C39.2, IC1.LO+
- net N$39: now also C157.1, IC29.OUT+, L40.2; no longer C42.1, IC1.OUT+, L6.2
- net N$4: now also R45.1, R48.1, R49.2, R52.2; no longer R123.1, R124.2, R6.1, R89.2
- net N$40: now also C160.1, IC29.OUT-, L41.2; no longer C55.1, IC1.OUT-, L12.2
- net N$41: now also C155.2, IC29.VSET, R84.1, R87.2; no longer C216.2, IC1.VSET, R115.1, R25.2
- net N$42: now also C134.2, IC27.LO-; no longer C45.2, IC6.LO-
- net N$43: now also C137.1, IC27.OUT+, R80.2; no longer C46.1, IC6.OUT+, R27.2
- net N$44: now also C138.1, IC27.OUT-, R81.2; no longer C47.1, IC6.OUT-, R28.2
- net N$45: now also C150.1, IC28.+OUT, R83.1, R86.2; no longer C51.1, IC7.+OUT, R30.1, R31.2
- net N$46: now also C149.2, IC28.-OUT, R82.2, R85.2; no longer C50.2, IC7.-OUT, R29.2, R32.2
- net N$47: now also C157.2, C161.1, L42.1; no longer C42.2, C56.1, L13.1
- net N$48: now also C160.2, C161.2, L43.1; no longer C55.2, C56.2, L14.1
- net N$49: now also C165.2, L43.2, L45.1; no longer C57.2, L14.2, L16.1
- net N$5: now also R46.1, R50.1; no longer R7.1, R8.1
- net N$50: now also C165.1, L42.2, L44.1; no longer C57.1, L13.2, L15.1
- net N$51: now also C77.1, IC17.VCC, L26.2; no longer C154.1, IC27.VCC, L4.2
- net N$52: now also C135.2, IC27.LO+; no longer C59.2, IC6.LO+
- net N$53: now also C162.2, C163.1, IC31.AIN+, R88.1; no longer C60.1, C61.2, IC8.AIN+, R119.1
- net N$54: now also C163.2, C164.1, IC31.AIN-, R89.1; no longer C60.2, C62.1, IC8.AIN-, R120.1
- net N$55: now also C167.1, L44.2, R90.2, R91.2; no longer C58.1, L15.2, R37.2, R38.2
- net N$56: now also C167.2, L45.2, R90.1, R92.2; no longer C58.2, L16.2, R37.1, R39.2
- net N$57: now also C43.1, L14.2, L18.1; no longer C222.1, L19.1, L20.2
- net N$58: now also C138.2, C150.2, IC28.-IN, R83.2; no longer C47.2, C51.2, IC7.-IN, R30.2
- net N$59: now also C137.2, C149.1, IC28.+IN, R82.1; no longer C46.2, C50.1, IC7.+IN, R29.1
- net N$6: now also C99.1, J2.1; no longer C1.1, J1.1
- net N$60: now also C39.2; no longer C65.2
- net N$61: now also C170.2; no longer C66.2
- net N$62: now also C130.1, L36.2, R63.2, R64.2; no longer C32.1, L9.2, R33.2, R34.2
- net N$63: now also C130.2, L37.2, R63.1, R65.2; no longer C32.2, L10.2, R33.1, R35.2
- net N$64: now also C67.2, IC10.TUNE, R15.2; no longer C118.2, IC14.TUNE, R50.2
- net N$66: now also C178.2, IC33.IN+; no longer C67.2, IC5.IN+
- net N$67: now also C179.2, IC33.IN-; no longer C68.2, IC5.IN-
- net N$68: now also C176.1, C179.1; no longer C68.1, C69.1
- net N$69: now also C176.2, C178.1; no longer C67.1, C69.2
- net N$7: now also C109.2, IC24.IN+; no longer C3.2, IC37.IN+
- net N$70: now also C185.1, IC33.LO-; no longer C70.1, IC5.LO-
- net N$71: now also C183.2, IC33.LO+; no longer C71.2, IC5.LO+
- net N$72: now also C191.1, IC33.OUT+, L46.2; no longer C74.1, IC5.OUT+, L21.2
- net N$73: now also C192.1, IC33.OUT-, L47.2; no longer C87.1, IC5.OUT-, L22.2
- net N$74: now also C186.2, IC33.VSET, R100.1, R101.2; no longer C220.2, IC5.VSET, R116.1, R41.2
- net N$75: now also C199.2, IC36.LO-; no longer C77.2, IC10.LO-
- net N$76: now also C202.1, IC36.OUT+, R102.2; no longer C78.1, IC10.OUT+, R43.2
- net N$77: now also C203.1, IC36.OUT-, R103.2; no longer C79.1, IC10.OUT-, R44.2
- net N$78: now also C173.1, C202.2, IC32.+IN, R94.1; no longer C78.2, C82.1, IC11.+IN, R45.1
- net N$79: now also C174.2, C203.2, IC32.-IN, R95.2; no longer C79.2, C83.2, IC11.-IN, R46.2
- net N$8: now also C110.2, IC24.IN-; no longer C4.2, IC37.IN-
- net N$80: now also C174.1, IC32.+OUT, R95.1, R97.2; no longer C83.1, IC11.+OUT, R46.1, R47.2
- net N$81: now also C173.2, IC32.-OUT, R94.2, R96.2; no longer C82.2, IC11.-OUT, R45.2, R48.2
- net N$82: now also C191.2, C194.1, L48.1; no longer C74.2, C88.1, L23.1
- net N$83: now also C192.2, C194.2, L49.1; no longer C87.2, C88.2, L24.1
- net N$84: now also C196.2, L49.2, L51.1; no longer C89.2, L24.2, L26.1
- net N$85: now also C196.1, L48.2, L50.1; no longer C89.1, L23.2, L25.1
- net N$86: now also C197.1, IC36.IN+, L50.2, L52.1; no longer C90.1, IC10.IN+, L25.2, L27.1
- net N$87: now also C197.2, IC36.IN-, L51.2, L53.1; no longer C90.2, IC10.IN-, L26.2, L28.1
- net N$88: now also C200.2, IC36.LO+; no longer C91.2, IC10.LO+
- net N$89: now also C187.2, C188.1, IC35.AIN+, R98.1; no longer C92.1, C93.2, IC12.AIN+, R121.1
- net N$9: now also C107.1, C110.1; no longer C4.1, C5.1
- net N$90: now also C188.2, C189.1, IC35.AIN-, R99.1; no longer C92.2, C94.1, IC12.AIN-, R122.1
- net N$91: now also C40.1, L11.2, L15.1; no longer C98.1, L32.1, L33.2
- net N$92: now also C101.2, C113.2, IC23.-IN, R56.2; no longer C21.2, C25.2, IC3.-IN, R18.2
- net N$93: now also C63.1, C66.1, IC10.CP_OUT, R15.1; no longer C117.1, C119.1, IC14.CP_OUT, R50.1
- net N$94: now also C58.1, IC10.REG; no longer C114.1, IC14.REG
- net N$95: now also C100.2, C112.1, IC23.+IN, R55.1; no longer C20.2, C24.1, IC3.+IN, R17.1
- net N$96: now also C41.1, L12.2, L16.1; no longer C101.1, L34.1, L35.2
- net N$97: now also C36.1, IC7.CLK1, L12.1; no longer C102.1, IC13.CLK1, L35.1
- net N$98: now also C59.1, IC10.NOISE_FILT; no longer C115.1, IC14.NOISE_FILT
- net N$99: now also C42.1, L13.2, L17.1; no longer C111.1, L36.1, L37.2
- net NRST: now also IC37.PG10-NRST, JP1.9; no longer IC9.PG10-NRST, JP2.9
- net OUT+: now also C121.1, R58.1, R61.2; no longer C27.1, R117.2, R20.1
- net OUT+1: now also C158.1, R85.1, R88.2; no longer C53.1, R119.2, R32.1
- net OUT+2: now also C184.1, R96.1, R98.2; no longer C85.1, R121.2, R48.1
- net OUT-: now also C121.2, R59.1, R62.2; no longer C27.2, R118.2, R19.1
- net OUT-1: now also C158.2, R86.1, R89.2; no longer C53.2, R120.2, R31.1
- net OUT-2: now also C184.2, R97.1, R99.2; no longer C85.2, R122.2, R47.1
- net OUT_CM: now also C116.1, IC23.VOCM; no longer C26.1, IC3.VOCM
- net OUT_CM1: now also C153.1, IC28.VOCM; no longer C52.1, IC7.VOCM
- net OUT_CM2: now also C182.1, IC32.VOCM; no longer C84.1, IC11.VOCM
- net PORT1LO1: now also C114.1, IC21.RFOUTA_N, R33.1; no longer C7.1, IC19.RFOUTA_N, R62.1
- net PORT1LO2: now also C46.1, C98.1, L17.2; no longer C103.1, C15.1, L36.2
- net PORT1MIX1_EN: now also IC24.ENBL, R130.1; no longer IC37.ENBL, R133.1
- net PORT1MIX2_EN: now also IC22.EN, IC23.SHDN, R131.2; no longer IC2.EN, IC3.SHDN, R134.2
- net PORT1SRC: now also C96.1, IC18.RF1; no longer C2.1, IC26.RF1
- net PORT1SWITCH: now also IC18.CTL1; no longer IC26.CTL1
- net PORT1_CONVSTART: now also IC26.CONVST; no longer IC4.CONVST
- net PORT1_SCLK: now also IC26.SCLK; no longer IC4.SCLK
- net PORT1_SDO: now also IC26.SDO; no longer IC4.SDO
- net PORT2LO1: now also C151.1, IC21.RFOUTB_P, R34.1; no longer C39.1, IC19.RFOUTB_P, R65.1
- net PORT2LO2: now also C135.1, C44.1, L15.2; no longer C59.1, C97.1, L32.2
- net PORT2MIX1_EN: now also IC29.ENBL, R121.1; no longer IC1.ENBL, R112.1
- net PORT2MIX2_EN: now also IC27.EN, IC28.SHDN, R122.2; no longer IC6.EN, IC7.SHDN, R111.2
- net PORT2SRC: now also C133.1, IC17.RF_COM; no longer C34.1, IC27.RF_COM
- net PORT2SWITCH: now also IC17.CTL1; no longer IC27.CTL1
- net PORT2_CONVSTART: now also IC31.CONVST; no longer IC8.CONVST
- net PORT2_SCLK: now also IC31.SCLK, R124.1; no longer IC8.SCLK, R135.1
- net PORT2_SDO: now also IC31.SDO, R123.1; no longer IC8.SDO, R136.1
- net PORTSWITCH1: now also IC16.CTL2; no longer IC25.CTL2
- net PORTSWITCH2: now also IC16.CTL1; no longer IC25.CTL1
- net REFLO1: now also C183.1, IC21.RFOUTA_P, R32.1; no longer C71.1, IC19.RFOUTA_P, R63.1
- net REFLO2: now also C200.1, C45.1, L16.2; no longer C100.1, C91.1, L34.2
- net REFLO3: now also C47.1, L18.2, R7.1, R8.1; no longer C221.1, L19.2, R73.1, R74.1
- net REFMIX1_EN: now also IC33.ENBL; no longer IC5.ENBL
- net REFMIX2_EN: now also IC32.SHDN, IC36.EN, R133.2; no longer IC10.EN, IC11.SHDN, R113.2
- net REFSRC: now also C170.1, R27.1, R28.2; no longer C66.1, R71.1, R72.2
- net REF_CONVSTART: now also IC35.CONVST; no longer IC12.CONVST
- net REF_SCLK: now also IC35.SCLK; no longer IC12.SCLK
- net REF_SDO: now also IC35.SDO; no longer IC12.SDO
- net SCL: now also IC2CONTROL.SCL, IC37.PC4, IC7.SCL, R116.1; no longer IC13.SCL, IC9.PC4, R90.1
- net SDA: now also IC2CONTROL.SDA, IC37.PA8, IC7.SDA, R117.1; no longer IC13.SDA, IC9.PA8, R95.1
- net SOURCE_CE: now also IC10.CE, R11.2; no longer IC14.CE, R56.2
- net SOURCE_CLK: now also IC10.CLK; no longer IC14.CLK
- net SOURCE_HIGHBAND: now also C68.2, IC13.RF1; no longer C121.2, IC22.RF1
- net SOURCE_LD: now also IC10.LD; no longer IC14.LD
- net SOURCE_LE: now also IC10.LE; no longer IC14.LE
- net SOURCE_LOWBAND: now also C48.1, IC13.RF2; no longer C157.1, IC22.RF2
- net SOURCE_MOSI: now also IC10.DATA; no longer IC14.DATA
- net SOURCE_MUX: now also IC10.MUX; no longer IC14.MUX
- net SOURCE_REF: now also C51.1, IC7.CLK3; no longer C130.1, IC13.CLK3
- net SOURCE_RF_EN: now also IC10.RFOUT_EN; no longer IC14.RFOUT_EN
- net SOURCE_VCC: now also C57.1, IC10.VCC_CP, IC10.VCC_PLL, IC11.VDD, IC12.VDD, L20.2, TP13.TP; no longer C128.1, IC14.VCC_CP, IC14.VCC_PLL, IC16.VDD, IC18.VDD, L39.2, TP17.TP
- net SWCLK: now also IC37.PA14, JP1.6; no longer IC9.PA14, JP2.6
- net SWDIO: now also IC37.PA13, JP1.8; no longer IC9.PA13, JP2.8
- net TCK: now also JP1.1; no longer JP2.1
- net TDI: now also JP1.3; no longer JP2.3
- net TDO: now also JP1.2; no longer JP2.2
- net TMS: now also JP1.4; no longer JP2.4
- net UART_TX: now also IC37.PC10, JP1.10; no longer IC9.PC10, JP2.10
- net VCCINT: now also C10.1, C213.1, C215.1, C217.1, C219.1, C7.1, IC2BUCK1.FB, L2.2; no longer C167.1, C169.1, C172.1, C179.1, C208.1, C209.1, C210.1, L53.2, R84.2
Other:
- note added: "I2C address: 0x42"
- note added: "I2C address: 0xC0"
- note removed: "Regulators on with floating enable"
- note removed: "Resistor set for 1MHz"
