File: Hardware/VNA.sch (EAGLE design)
At the start: 503 parts, among them IC1 MIC2253, IC10 MAX2871, IC11 RFSW6042, IC12 RFSW6042, IC13 QPC6324, IC14 RFSA3714, IC15 TRF37A73, IC16 QPC6324, IC17 QPC6324, IC18 QPC6324, IC19 AP2114H, IC2 LM3370SD-4221, IC20 NCP702-3.3, IC21 MAX2871, IC22 LT5560, IC23 THS4521IDGKR, IC24 ADL5801, IC25 NCP702-1.8, IC26 MCP33131D-10-E/MS, IC27 LT5560, IC28 THS4521IDGKR, IC29 ADL5801, IC3 LDL212PU50R, IC30 NCP702-1.8, IC31 MCP33131D-10-E/MS, IC32 THS4521IDGKR, IC33 ADL5801, IC34 NCP702-1.8, IC35 MCP33131D-10-E/MS, IC36 LT5560, IC37 STM32G431CB, IC4 LDL212PU50R, IC5 LDL212PU50R, IC6 LDL212PU50R, IC7 SI5351C, IC8 AP2114H, IC9 NCP702-3.3, J1 PJ-014D, J2 AMPHENOL_132289, J3 AMPHENOL_132289, J4 TYPE-C16P(073), Q1 SSM3J338R, Q2 SSM3J338R, T1 B012-617DB-1-63-B331, T2 B012-617DB-1-63-B331, T3 B012-617DB-1-63-B331, U1 W25Q16BVSN, U2 6SLX9TQG144, X1 SMA_CONNECTOR, X2 SMA_CONNECTOR, Y1 DSB221SDN/26MHz

Commit message: Additional filters for digital control lines, attenuator for Port1/Ref 1.LO
Parts:
- removed L11, L12, L13, L15, L16, L17: 120n, VNA:INDUCTOR0402
- added C223, C224, C225, C226, C227, C228, C229, C230, C231, C232, C233, C234, C235, C236, C237, C238, C239, C240, C241, C242, C243, C244, C245, C246, C247, C248, C249, C250, C251, C252, C253, C254, C255, C256, C257, C258, C259, C260, C261, C262, C263, C264, C265, C266, C267, C268, C271, C272, C273, C274: 100p, VNA:C-EUC0402:2
- added C269, C270: 100n, VNA:C-EUC0402:2
- added R143, R144, R145, R146, R147, R148, R149, R150, R151, R152, R153, R154, R155, R156, R157, R158, R159, R160, R161, R162, R163, R165, R166: 10k, VNA:R-EU_R0402
- added R164, R167, R169, R170, R171, R172, R174, R175: 100, VNA:R-EU_R0402
- added R168, R173: 75, VNA:R-EU_R0402
- added R176, R177, R178, R179, R180, R181: 0, VNA:R-EU_R0402
- C35, C36, C37, C44, C45, C46: value 18p -> DNP
- C40, C41, C42: value 56p -> DNP
Connections:
- new net N$169: C225.1, R132.1, R144.1, U2B0.IO_L1P_HSWAPEN_0
- new net N$170: C227.1, R131.2, R145.2, U2B0.IO_L3P_0
- new net N$172: C232.1, R122.2, R147.1, U2B2.IO_L14N_D12_2
- new net N$173: C229.1, R130.1, R146.1, U2B0.IO_L2N_0
- new net N$174: C236.1, IC17.CTL1, R149.1
- new net N$176: C240.1, IC16.CTL2, R151.1
- new net N$178: C238.1, IC16.CTL1, R150.1
- new net N$180: C268.1, IC10.CE, R163.1
- new net N$182: C242.1, IC18.CTL1, R152.1
- new net N$184: C244.1, IC15.PWDN, R153.1
- new net N$185: C246.1, IC13.CTL1, R154.1
- new net N$192: C250.1, IC14.D0, R156.1
- new net N$193: C248.1, IC13.CTL2, R155.1
- new net N$226: IC10.CLK, R164.1
- new net N$227: C252.1, IC14.D1, R157.1
- new net N$232: IC10.DATA, R170.1
- new net N$257: C254.1, IC14.D2, R158.1
- new net N$258: IC10.LE, R171.1
- new net N$259: C256.1, IC14.D3, R159.1
- new net N$260: C257.1, IC14.D6, R160.2
- new net N$261: IC10.MUX, R167.1
- new net N$262: C259.1, IC14.D5, R161.2
- new net N$263: C272.1, IC10.RFOUT_EN, R165.1
- new net N$264: C261.1, IC14.D4, R162.2
- new net N$265: C269.2, R168.2, R172.1
- new net N$266: C274.1, IC10.LD, R166.1
- new net N$267: C114.1, R168.1, R169.1
- new net N$268: C270.2, R173.2, R175.1
- new net N$269: C183.1, R173.1, R174.1
- new net N$312: C223.1, R133.2, R143.2, U2B0.IO_L1N_VREF_0
- new net N$512: C234.1, R121.1, R148.2, U2B2.IO_L14P_D11_2
- net AMP_PWDN: now also C243.1, R153.2; no longer IC15.PWDN
- net ATT_D0: now also C249.1, R156.2; no longer IC14.D0
- net ATT_D1: now also C251.1, R157.2; no longer IC14.D1
- net ATT_D2: now also C253.1, R158.2; no longer IC14.D2
- net ATT_D3: now also C255.1, R159.2; no longer IC14.D3
- net ATT_D4: now also C262.1, R162.1; no longer IC14.D4
- net ATT_D5: now also C260.1, R161.1; no longer IC14.D5
- net ATT_D6: now also C258.1, R160.1; no longer IC14.D6
- net FILT_IN_C1: now also C263.1
- net FILT_IN_C2: now also C264.1
- net FILT_OUT_C1: now also C266.1
- net FILT_OUT_C2: now also C265.1
- net GND: now also C223.2, C224.2, C225.2, C226.2, C227.2, C228.2, C229.2, C230.2, C231.2, C232.2, C233.2, C234.2, C235.2, C236.2, C237.2, C238.2, C239.2, C240.2, C241.2, C242.2, C243.2, C244.2, C245.2, C246.2, C247.2, C248.2, C249.2, C250.2, C251.2, C252.2, C253.2, C254.2, C255.2, C256.2, C257.2, C258.2, C259.2, C260.2, C261.2, C262.2, C263.2, C264.2, C265.2, C266.2, C267.2, C268.2, C271.2, C272.2, C273.2, C274.2, R169.2, R172.2, R174.2, R175.2
- net HIGHBAND_SELECT: now also C245.1, R154.2; no longer IC13.CTL1
- net LOWBAND_SELECT: now also C247.1, R155.2; no longer IC13.CTL2
- net N$101: now also R180.1; no longer L11.1
- net N$160: now also R176.1; no longer L13.1
- net N$91: now also R180.2, R181.1; no longer L11.2, L15.1
- net N$96: now also R178.1, R179.2; no longer L12.2, L16.1
- net N$97: now also R179.1; no longer L12.1
- net N$99: now also R176.2, R177.1; no longer L13.2, L17.1
- net PORT1LO1: now also C269.1; no longer C114.1
- net PORT1LO2: now also R177.2; no longer L17.2
- net PORT1MIX1_EN: now also C230.1, R146.2; no longer R130.1, U2B0.IO_L2N_0
- net PORT1MIX2_EN: now also C228.1, R145.1; no longer R131.2, U2B0.IO_L3P_0
- net PORT1SWITCH: now also C241.1, R152.2; no longer IC18.CTL1
- net PORT2LO2: now also R181.2; no longer L15.2
- net PORT2MIX1_EN: now also C233.1, R148.1; no longer R121.1, U2B2.IO_L14P_D11_2
- net PORT2MIX2_EN: now also C231.1, R147.2; no longer R122.2, U2B2.IO_L14N_D12_2
- net PORT2SWITCH: now also C235.1, R149.2; no longer IC17.CTL1
- net PORTSWITCH1: now also C239.1, R151.2; no longer IC16.CTL2
- net PORTSWITCH2: now also C237.1, R150.2; no longer IC16.CTL1
- net REFLO1: now also C270.1; no longer C183.1
- net REFLO2: now also R178.2; no longer L16.2
- net REFMIX1_EN: now also C226.1, R144.2; no longer R132.1, U2B0.IO_L1P_HSWAPEN_0
- net REFMIX2_EN: now also C224.1, R143.1; no longer R133.2, U2B0.IO_L1N_VREF_0
- net SOURCE_CE: now also C267.1, R163.2; no longer IC10.CE
- net SOURCE_CLK: now also R164.2; no longer IC10.CLK
- net SOURCE_LD: now also C273.1, R166.2; no longer IC10.LD
- net SOURCE_LE: now also R171.2; no longer IC10.LE
- net SOURCE_MOSI: now also R170.2; no longer IC10.DATA
- net SOURCE_MUX: now also R167.2; no longer IC10.MUX
- net SOURCE_RF_EN: now also C271.1, R165.2; no longer IC10.RFOUT_EN
Other:
- note removed: "3x110MHz lowpass"
- note removed: "CTL2 low: RF_COM->RF1 CTL2 high: RF_COM->RF2"
- moved on the sheet: C209, C210, C211, C212, C213, C214, C215, C216, C217, C218, C219, C220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
