File: Hardware/Experiments/SynthEvaluationBoard.brd (EAGLE design)
At the start: 100 x 100 mm, 174 parts, among them IC1 STW81200, IC19 AP2114H, IC2 AD9913, IC3 NCP702-1.8, IC34 NCP702-1.8, IC4 SI5332A-GM1, IC5 STM32L462CE, J1 AMPHENOL_901-10510-2, J2 AMPHENOL_901-10510-2, J3 AMPHENOL_901-10510-2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

Commit message: Minor adjustments + gerbers
Parts:
- added LED1, LED2, LED3, LED4, LED5: Green, eagle-ltspice:LED_SML0603
- added R52: 470, VNA:R0402
- added R53, R54, R55, R56: 220, VNA:R0402
- R46: value 10k -> 1k
Connections:
- new net N$48: LED3.A, R52.1
- new net N$50: LED1.A, R53.1
- new net N$52: LED2.A, R54.1
- new net N$53: LED4.A, R55.1
- new net N$65: LED5.A, R56.1
- new net N$81: IC5.13, R53.2
- new net N$82: IC5.12, R54.2
- new net N$83: IC5.11, R55.2
- new net N$84: IC5.10, R56.2
- net +5V: now also R52.2
- net GND: now also LED1.C, LED2.C, LED3.C, LED4.C, LED5.C
Routing:
- net +5V: track 14.8 -> 25.4 mm
- net GND: track 108.5 -> 114.7 mm, vias 1590 -> 1674
- net N$81: track 0.00 -> 5.83 mm
- net N$82: track 0.00 -> 5.35 mm
- net N$83: track 0.00 -> 4.35 mm
- net N$84: track 0.00 -> 3.52 mm
- net N$65: track 0.00 -> 1.69 mm
- net N$53: track 0.00 -> 1.69 mm
- net N$52: track 0.00 -> 1.69 mm
- net N$50: track 0.00 -> 1.69 mm
- net N$48: track 0.00 -> 1.69 mm
Other:
- board text added: "Hardware/Experiments/SynthEvaluationBoard"
- board text added: "LED1"
- board text added: "LED2"
- board text added: "LED3"
- board text added: "LED4"
- board text added: "github.com/jankae/LibreVNA"

Commit message: Added milling layer to gerber, created BOM
Parts:
- R23, R24: value (none) -> 49R9
Changed lines of the file:
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@@
 </element>
 <element name="J1" library="VNA" library_urn="urn:adsk.eagle:library:22367181" package="AMPHENOL_901-10510-2" value="AMPHENOL_901-10510-2" x="17.9" y="100" smashed="yes" rot="R90"/>
-<element name="R23" library="VNA" library_urn="urn:adsk.eagle:library:22367181" package="R0402" package3d_urn="urn:adsk.eagle:package:22367274/3" value="" x="17.9" y="92" smashed="yes" rot="R90">
+<element name="R23" library="VNA" library_urn="urn:adsk.eagle:library:22367181" package="R0402" package3d_urn="urn:adsk.eagle:package:22367274/3" value="49R9" x="17.9" y="92" smashed="yes" rot="R90">
 <attribute name="NAME" x="17.265" y="91.365" size="1.27" layer="25" rot="R90"/>
 <attribute name="VALUE" x="19.805" y="91.365" size="1.27" layer="27" rot="R90"/>
@@
 <attribute name="VALUE" x="51.89" y="1.27" size="1.778" layer="27" rot="R90"/>
 </element>
-<element name="R24" library="VNA" library_urn="urn:adsk.eagle:library:22367181" package="R0402" package3d_urn="urn:adsk.eagle:package:22367274/3" value="" x="19" y="7" smashed="yes" rot="R270">
+<element name="R24" library="VNA" library_urn="urn:adsk.eagle:library:22367181" package="R0402" package3d_urn="urn:adsk.eagle:package:22367274/3" value="49R9" x="19" y="7" smashed="yes" rot="R270">
 <attribute name="NAME" x="19.635" y="7.635" size="1.27" layer="25" rot="R270"/>
 <attribute name="VALUE" x="17.095" y="7.635" size="1.27" layer="27" rot="R270"/>

Commit message: minimal working Si5332/AD9913
Parts:
- R29: value 49R9 -> 4k64
Changed lines of the file:
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@@
 <attribute name="VALUE" x="70.0091" y="76.9" size="1.27" layer="27" rot="R270" align="top-center"/>
 </element>
-<element name="R29" library="VNA" library_urn="urn:adsk.eagle:library:22367181" package="R0402" package3d_urn="urn:adsk.eagle:package:22367274/3" value="49R9" x="75.9" y="71.9" smashed="yes" rot="R90">
+<element name="R29" library="VNA" library_urn="urn:adsk.eagle:library:22367181" package="R0402" package3d_urn="urn:adsk.eagle:package:22367274/3" value="4k64" x="75.9" y="71.9" smashed="yes" rot="R90">
 <attribute name="NAME" x="75.265" y="71.265" size="1.27" layer="25" rot="R90"/>
 <attribute name="VALUE" x="77.805" y="71.265" size="1.27" layer="27" rot="R90"/>
