File: Hardware/Kicad/FPGAMicrocontroller.kicad_sch (KiCad schematic)
At the start: 26 parts, among them IC37 STM32G431CB, J4 USB_C_Receptacle_USB2.0_16P, U1 W25Q16BVSN

Commit message: Swapped LED1 and LED2
1) Swapped LED1 and LED2 identifiers to be consistent with original schematic and correct color in BOM
Parts:
- renumbered LED2 to LED1
Connections:
- net LED2C renamed LED1C
Changed lines of the file:
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@@
 		)
 	)
-	(label "LED2C"
+	(label "LED1C"
 		(at 222.25 121.92 90)
 		(fields_autoplaced yes)
@@
 		(dnp no)
 		(fields_autoplaced yes)
-		(property "Reference" "LED2"
+		(property "Reference" "LED1"
 			(at 226.06 115.8874 90)
 			(effects
@@
 			(project "VNA"
 				(path "/7469840a-34dd-443e-8d3c-7bb0beac8ed2/5d6d43e6-b4b8-4453-a605-266bbc2eda13"
-					(reference "LED2")
+					(reference "LED1")
 					(unit 1)
 				)
