File: Hardware/Kicad/VNA.kicad_sch (KiCad schematic)
At the start: 2 parts

Commit message: Removed Unused vias per DRC  [Net-(IC34-EN)], [PORTSW2_CTL_F], [PORTSW1_CTL_F], [Net-(IC30-EN)] Reverted Soldermask Extension for top cover plate Regenerated Gerbers
Other:
- moved on the sheet: N1, N2
Changed lines of the file:
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@@
 	(symbol
 		(lib_id "Mechanical:Housing")
-		(at 52.07 147.32 0)
+		(at 27.94 144.78 0)
 		(unit 1)
 		(exclude_from_sim no)
@@
 		(fields_autoplaced yes)
 		(property "Reference" "N1"
-			(at 55.88 146.3674 0)
+			(at 31.75 143.8274 0)
 			(effects
 				(font
@@
 		)
 		(property "Value" "Top Cover"
-			(at 55.88 148.9074 0)
+			(at 31.75 146.3674 0)
 			(effects
 				(font
@@
 		)
 		(property "Footprint" "VNA:VNA_COVER_TOP"
-			(at 53.34 146.05 0)
+			(at 29.21 143.51 0)
 			(effects
 				(font
@@
 		)
 		(property "Datasheet" "~"
-			(at 53.34 146.05 0)
+			(at 29.21 143.51 0)
 			(effects
 				(font
@@
 		)
 		(property "Description" "Housing"
-			(at 52.07 147.32 0)
+			(at 27.94 144.78 0)
 			(effects
 				(font
@@
 	(symbol
 		(lib_id "Mechanical:Housing")
-		(at 52.07 158.75 0)
+		(at 49.53 144.78 0)
 		(unit 1)
 		(exclude_from_sim no)
@@
 		(fields_autoplaced yes)
 		(property "Reference" "N2"
-			(at 55.88 157.7974 0)
+			(at 53.34 143.8274 0)
 			(effects
 				(font
@@
 		)
 		(property "Value" "Bottom Cover"
-			(at 55.88 160.3374 0)
+			(at 53.34 146.3674 0)
 			(effects
 				(font
@@
 		)
 		(property "Footprint" "VNA:VNA_COVER_BOTTOM"
-			(at 53.34 157.48 0)
+			(at 50.8 143.51 0)
 			(effects
 				(font
@@
 		)
 		(property "Datasheet" "~"
-			(at 53.34 157.48 0)
+			(at 50.8 143.51 0)
 			(effects
 				(font
@@
 		)
 		(property "Description" "Housing"
-			(at 52.07 158.75 0)
+			(at 49.53 144.78 0)
 			(effects
 				(font
