File: Hardware/Kicad/LocalOsc2_RefClock.kicad_sch (KiCad schematic)
At the start: 37 parts, among them IC7 SI5351C, X1 SMA, X2 SMA, Y1 26MHz

Commit message: Production files
Production files as sent to fabricator.
 Includes various PCB cleanup an the TCXO footprint change due to an unavailable part.
Parts:
- Y1: footprint VNA:2.5X2.0_KXO-86-TCXO -> VNA:Oscillator_SMD_ECS_20CSMV4_2.0x1.6mm; MPN DSB221SDN/26MHz -> ECS-TXO-20CSMV4-260-AN-TR
Changed lines of the file:
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@@
+		(length 2.54)
+		(shape round)
+		(at 180.34 154.94 0)
+		(fields_autoplaced yes)
+		(effects
+			(font
+				(size 1.27 1.27)
+			)
+			(justify left bottom)
+		)
+		(property "Netclass" "RF"
+			(at 181.0385 152.4 0)
+			(effects
+				(font
+					(size 1.27 1.27)
+					(italic yes)
+				)
+				(justify left)
+			)
+		)
+	)
+	(netclass_flag ""
 		(length 2.54)
 		(shape round)
@@
 		(length 2.54)
 		(shape round)
-		(at 297.18 193.04 0)
+		(at 180.34 139.7 0)
 		(fields_autoplaced yes)
 		(effects
@@
 		)
 		(property "Netclass" "RF"
+			(at 181.0385 137.16 0)
+			(effects
+				(font
+					(size 1.27 1.27)
+					(italic yes)
+				)
+				(justify left)
+			)
+		)
+	)
+	(netclass_flag ""
+		(length 2.54)
+		(shape round)
+		(at 180.34 165.1 0)
+		(fields_autoplaced yes)
+		(effects
+			(font
+				(size 1.27 1.27)
+			)
+			(justify left bottom)
+		)
+		(property "Netclass" "RF"
+			(at 181.0385 162.56 0)
+			(effects
+				(font
+					(size 1.27 1.27)
+					(italic yes)
+				)
+				(justify left)
+			)
+		)
+	)
+	(netclass_flag ""
+		(length 2.54)
+		(shape round)
+		(at 180.34 129.54 0)
+		(fields_autoplaced yes)
+		(effects
+			(font
+				(size 1.27 1.27)
+			)
+			(justify left bottom)
+		)
+		(property "Netclass" "RF"
+			(at 181.0385 127 0)
+			(effects
+				(font
+					(size 1.27 1.27)
+					(italic yes)
+				)
+				(justify left)
+			)
+		)
+	)
+	(netclass_flag ""
+		(length 2.54)
+		(shape round)
+		(at 180.34 149.86 0)
+		(fields_autoplaced yes)
+		(effects
+			(font
+				(size 1.27 1.27)
+			)
+			(justify left bottom)
+		)
+		(property "Netclass" "RF"
+			(at 181.0385 147.32 0)
+			(effects
+				(font
+					(size 1.27 1.27)
+					(italic yes)
+				)
+				(justify left)
+			)
+		)
+	)
+	(netclass_flag ""
+		(length 2.54)
+		(shape round)
+		(at 297.18 193.04 0)
+		(fields_autoplaced yes)
+		(effects
+			(font
+				(size 1.27 1.27)
+			)
+			(justify left bottom)
+		)
+		(property "Netclass" "RF"
 			(at 297.8785 190.5 0)
+			(effects
+				(font
+					(size 1.27 1.27)
+					(italic yes)
+				)
+				(justify left)
+			)
+		)
+	)
+	(netclass_flag ""
+		(length 2.54)
+		(shape round)
+		(at 180.34 134.62 0)
+		(fields_autoplaced yes)
+		(effects
+			(font
+				(size 1.27 1.27)
+			)
+			(justify left bottom)
+		)
+		(property "Netclass" "RF"
+			(at 181.0385 132.08 0)
 			(effects
 				(font
@@
 		(property "Netclass" "RF"
 			(at 83.2485 139.7 0)
+			(effects
+				(font
+					(size 1.27 1.27)
+					(italic yes)
+				)
+				(justify left)
+			)
+		)
+	)
+	(netclass_flag ""
+		(length 2.54)
+		(shape round)
+		(at 180.34 160.02 0)
+		(fields_autoplaced yes)
+		(effects
+			(font
+				(size 1.27 1.27)
+			)
+			(justify left bottom)
+		)
+		(property "Netclass" "RF"
+			(at 181.0385 157.48 0)
 			(effects
 				(font
@@
 			)
 		)
-		(property "Footprint" "VNA:2.5X2.0_KXO-86-TCXO"
+		(property "Footprint" "VNA:Oscillator_SMD_ECS_20CSMV4_2.0x1.6mm"
 			(at 99.568 103.632 0)
 			(effects
@@
 			)
 		)
-		(property "Datasheet" "https://www.geyer-electronic.de/wp-content/uploads/2022/09/GEYER-KXO-86-TCXO-HCMOS.pdf"
+		(property "Datasheet" "https://ecsxtal.com/store/pdf/ECS-TXO-20CSMV4.pdf"
 			(at 99.06 116.84 0)
 			(effects
@@
 			)
 		)
-		(property "MPN" "DSB221SDN/26MHz"
+		(property "MPN" "ECS-TXO-20CSMV4-260-AN-TR"
 			(at 99.06 116.84 0)
 			(effects
