File: Hardware/Kicad/PowerSupply.kicad_sch (KiCad schematic)
At the start: 65 parts, among them IC1 MIC2253, IC2 LM3370, IC3 LDL212PU50R, IC4 LDL212PU50R, IC5 LDL212PU50R, IC6 LDL212PU50R, J1 PJ-014D, Q1 SSM3J338R, Q2 SSM3J338R

Commit message: Removed Unused vias per DRC  [Net-(IC34-EN)], [PORTSW2_CTL_F], [PORTSW1_CTL_F], [Net-(IC30-EN)] Reverted Soldermask Extension for top cover plate Regenerated Gerbers
Parts:
- D1: footprint Diode_SMD_AKL:D_SMB -> Diode_SMD:D_SMB
Changed lines of the file:
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@@
 			)
 		)
-		(property "Footprint" "Diode_SMD_AKL:D_SMB"
+		(property "Footprint" "Diode_SMD:D_SMB"
 			(at 116.84 104.14 0)
 			(effects

Commit message: change LM3370 MPN to LM3370SD-3021(defualt 1.2v for buck 1)
Parts:
- IC2: MPN LM3370SD-4221 -> LM3370SD-3021
Changed lines of the file:
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@@
 			)
 		)
-		(property "MPN" "LM3370SD-4221"
+		(property "MPN" "LM3370SD-3021"
 			(at 101.6 190.5 0)
 			(effects
@@
 			)
 		)
-		(property "MPN" "LM3370SD-4221"
+		(property "MPN" "LM3370SD-3021"
 			(at 101.6 231.14 0)
 			(effects
@@
 			)
 		)
-		(property "MPN" "LM3370SD-4221"
+		(property "MPN" "LM3370SD-3021"
 			(at 208.28 180.34 0)
 			(effects
